File: bioshield.brd (EAGLE design)
At the start: 68.6 x 53.3 mm, 10 parts

Commit message: Schematic nearly complete
Parts:
- removed JP1: (no value), pinhead:1X01
- removed JP2: (no value), pinhead:1X05
- removed RESET: (no value), switch-omron:B3F-10XX
- added C1, C20, C21, C22, C23, C24, C29, C32, C33, C34, C35, C36, C37, C38, C5, C6, C7: (no value), SparkFun-Capacitors:CAP-PTH-5MM
- added C10: 22pF, SparkFun-Passives:CAP-PTH-5MM
- added C11, C12, C3: 100nF, SparkFun-Passives:CAP-PTH-5MM
- added C13: 10uF, SparkFun-Passives:CAP-PTH-5MM
- added C14: 10nF, SparkFun-Passives:CAP-PTH-5MM
- added C15: 1uF, SparkFun-Passives:CAP-PTH-5MM
- added C16: 4.3uF, SparkFun-Passives:CAP-PTH-5MM
- added C2: 3.2u, SparkFun-Passives:CAP-PTH-5MM
- added C4: 220nF, SparkFun-Passives:CAP-PTH-5MM
- added C8: 1uF, adafruit:E2-5
- added C9: 1nF, SparkFun-Passives:CAP-PTH-5MM
- added D1: 5.1V, SparkFun-DiscreteSemi:DIODE-ZENER
- added DIGITAL1, POWER: (no value), SmartPrj:1X08-TH
- added DIGITAL2: (no value), SmartPrj:1X10-TH
- added IC1, IC3, IC8: LMC660, adafruit:DIL14
- added IC10, IC11, IC12, IC13, IC2, IC4, IC6, IC7, IC9: QUAD_OPAMPP, adafruit:DIL14
- added IC14, IC15, IC5: 4066N, 40xx:DIL14
- added J7: HC-05/HC-06, pinhead:1X06
- added J8: ELECTRODES, SparkFun-Connectors:2X6
- added J9: POWER_JACKPTH, SparkFun-Connectors:POWER_JACK_PTH
- added R1, R4, R43, R54, R55, R56, R57, R6, R61, R62, R63, R64: 10K, adafruit:0204/5
- added R10, R11, R15, R17, R20, R21, R22, R24, R7, R8, R9: 50K, adafruit:0204/5
- added R100, R86, R87, R88, R91, R99: (no value), rcl:0207/10
- added R12, R2: 1M, adafruit:0204/5
- added R13: 5M, adafruit:0204/5
- added R14, R16, R18, R19, R23: 30K, adafruit:0204/5
- added R25, R69: (no value), resistor:0207/10
- added R26: 16K, adafruit:0204/5
- added R27: 18K, adafruit:0204/5
- added R28: 100K, adafruit:0204/5
- added R29: 120-320, adafruit:0204/5
- added R3: 40K, adafruit:0204/5
- added R30: 220K, adafruit:0204/5
- added R31: 160K, adafruit:0204/5
- added R32: 500K, adafruit:0204/5
- added R33: 1K-6K, adafruit:0204/5
- added R34: 2.4K, adafruit:0204/5
- added R35: 3.9K, adafruit:0204/5
- added R36, R37: 4.99K, adafruit:0204/5
- added R38, R39, R40, R41: 9.53K, adafruit:0204/5
- added R42: (no value), adafruit:0204/5
- added R5: 5.1K, adafruit:0204/5
- added R51, R52, R59, R60: 24.7K, adafruit:0204/5
- added R53, R58, R65: 1.3K, adafruit:0204/5
- added R66, R67, R68, R70, R71, R72, R78, R82, R83, R85, R92, R93, R94, R95, R96, R97, R98: (no value), adafruit:0207/10
- added SH1, SH2, SH3: SHORT, stanford_iot_research:R0OHM
- added T1, T2, T3, T4: 2N2222, adafruit:TO92-EBC-OVAL
- J2: device SmartPrj:1X08-TH -> pinhead:1X05
- J4: device SmartPrj:1X10-TH -> SmartPrj:1X08-TH
- J5: device SmartPrj:1X08-TH -> pinhead:1X01
- J6: value (none) -> FTDI/EZ-LINK; device SmartPrj:1X08-TH -> pinhead:1X06
- moved J6 504.8 mm to (-53.3, -491.0)
- moved J1 51.4 mm to (36.8, 2.54), turned to 0 degrees
- moved J5 42.8 mm to (63.5, 5.71), turned to 0 degrees
- moved J4 24.4 mm to (54.6, 47.6)
- moved J2 19.3 mm to (55.9, 5.71)
Connections:
- removed net +5V: J2.5, J6.5
- removed net GND: J2.6, J2.7, J6.6, J6.7, RESET.1, RESET.2
- removed net N$122: ANALOG.1, JP2.1
- new net 2KHZ_OSC: IC14.5, IC6.1, R27.2, R28.2, R43.1
- new net 30KHZ_OSC: C22.2, IC5.13, R66.1, T3.B
- new net ADC_ECG: ANALOG.2, IC2.8, IC2.9, J2.2
- new net ADC_ICG: ANALOG.4, IC2.1, IC2.2, J2.4
- new net ADC_PPG: ANALOG.1, IC2.13, IC2.14, J2.1
- new net ADC_RESP: ANALOG.3, IC2.6, IC2.7, J2.3
- new net AGND: C11.1, C12.1, C15.2, C23.2, C3.2, C32.1, C33.1, C37.2, C38.2, C9.2, IC1.12, IC12.10, IC5.4, IC7.3, J8.10, J8.12, J8.8, R10.1, R100.1, R2.1, R26.1, R31.1, R33.1, R4.1, R41.2, R57.2, R66.2, R68.1, R85.1, R86.1, R9.1, R92.1, R96.1, SH2.2, T3.E, T4.E
- new net AVCC: IC1.4, R25.2, R29.2, SH1.2
- new net AVSS: IC1.11, SH3.2
- new net CLOCK1: C22.1, IC12.1, R83.1, R87.2, R88.2
- new net DGND: C1.2, C5.2, C6.2, C7.2, D1.P$2, IC2.11, IC4.11, J1.6, J1.7, J6.1, J6.2, J7.3, J9.GND, POWER.6, POWER.7, R11.1, R15.1, R17.1, R21.1, R22.1, R24.1, SH3.1
- new net ECG_E1: J8.1, R7.1
- new net ECG_E2: J8.3, R8.1
- new net ECG_E3: J8.5, R12.2, R13.2
- new net ECG_OUT: C4.2, IC1.6, IC1.7, R18.1
- new net ELECTRODE3: C29.1, R78.1, R91.2
- new net ICG_DEMUX: IC12.14, R67.1, R72.2, R95.1
- new net ICG_E1: C20.1, J8.7
- new net ICG_E2: C21.1, J8.9
- new net ICG_E3: C29.2, J8.11
- new net ICG_OUT: C36.2, IC11.8, R14.1, R99.2
- new net N$10: IC4.1, T1.B
- new net N$100: IC12.5, R85.2, R91.1
- new net N$101: C24.2, IC12.9, R69.1
- new net N$102: IC12.12, R70.2, R72.1
- new net N$103: C35.1, IC11.6, R92.2, R93.1
- new net N$105: IC11.2, R96.2, R97.1
- new net N$106: C36.1, R94.2, R98.1
- new net N$107: C35.2, IC11.7, R93.2, R94.1
- new net N$108: C37.1, IC11.10, R98.2
- new net N$109: IC11.9, R100.2, R99.1
- new net N$11: C2.2, IC1.3, R2.2
- new net N$110: C23.1, C34.1, R67.2
- new net N$12: C3.1, IC1.5, R6.2
- new net N$13: IC1.1, R3.2, R5.1
- new net N$14: C4.1, R5.2, R6.1
- new net N$15: IC1.14, R13.1
- new net N$16: IC9.3, R8.2
- new net N$2: IC1.2, R3.1, R4.2
- new net N$23: C21.2, IC10.3, R10.2
- new net N$24: C24.1, IC12.8, R64.2
- new net N$25: IC10.2, R59.1, R65.1
- new net N$26: IC1.13, R12.1, R53.1, R58.2
- new net N$27: IC10.1, R59.2, R63.1
- new net N$28: C1.1, IC2.3, R14.2, R15.2
- new net N$29: C6.1, IC2.10, R18.2, R22.2
- new net N$3: C5.1, IC2.5, R16.2, R17.2
- new net N$30: C7.1, IC2.12, R23.2, R24.2
- new net N$32: C32.2, C33.2, IC12.2, R88.1
- new net N$33: IC4.2, R11.2, R19.1
- new net N$35: IC5.1, R71.2
- new net N$36: D1.P$1, IC4.3, R1.1
- new net N$37: IC12.13, IC5.2, IC5.3
- new net N$38: IC4.5, R20.1, R21.2
- new net N$40: C38.1, IC11.3, R95.2
- new net N$41: IC4.7, T2.B
- new net N$42: IC13.6, R38.2, R39.1
- new net N$47: IC9.2, R51.1, R58.1
- new net N$51: IC5.5, R25.1, T3.C
- new net N$53: C13.1, IC13.7, R39.2
- new net N$55: C9.1, IC6.2, R28.1
- new net N$57: IC6.3, R26.2, R27.1
- new net N$62: C10.1, IC14.4, IC15.4, IC7.1, R30.2
- new net N$64: C13.2, IC7.5, R31.2
- new net N$66: C14.2, IC7.6, R32.1, R33.2
- new net N$67: C14.1, IC7.7, R32.2, R34.1
- new net N$68: C16.1, R34.2, R35.1
- new net N$69: IC9.1, R51.2, R56.1
- new net N$70: IC9.5, R56.2, R57.1
- new net N$71: IC1.9, R52.1, R53.2
- new net N$72: IC1.8, R52.2, R54.1
- new net N$73: IC1.10, R7.2
- new net N$74: IC10.5, R63.2, R64.1
- new net N$75: IC9.6, R54.2, R55.1
- new net N$76: IC3.9, R60.1, R65.2
- new net N$77: C2.1, IC9.7, R55.2
- new net N$78: IC3.8, R60.2, R61.1
- new net N$79: C20.2, IC3.10, R9.2
- new net N$80: IC10.6, R61.2, R62.1
- new net N$81: C15.1, IC7.10, R35.2
- new net N$84: IC10.7, R62.2, R69.2, R70.1, R71.1
- new net N$95: IC12.6, R82.1, R83.2
- new net N$96: C34.2, IC11.5, R68.2
- new net N$97: IC12.3, R86.2, R87.1
- new net PPG_DP: C10.2, IC7.2, J8.6, R30.1
- new net PPG_IA_N: C11.2, IC13.3, IC15.3
- new net PPG_IA_P: C12.2, IC14.3, IC8.10
- new net PPG_LEDN: IC15.5, J8.4, T4.C
- new net PPG_LEDP: J8.2, R29.1
- new net PPG_OUT: C16.2, IC7.8, IC7.9, R23.1
- new net RESP_OUT: IC11.1, R16.1, R97.2
- new net RX: DIGITAL1.1, J4.1, J6.4, J7.4
- new net TX: DIGITAL1.2, J4.2, J6.5, J7.5
- new net V+: IC10.4, IC11.4, IC12.4, IC12.7, IC13.4, IC3.4, IC6.4, IC7.4, IC8.4, IC9.4, R78.2, R82.2
- new net V-: IC10.11, IC11.11, IC12.11, IC13.11, IC3.11, IC6.11, IC7.11, IC8.11, IC9.11
- new net VCC_4V: IC4.6, SH2.1, T2.E
- new net VCC_5V: DIGITAL2.8, IC2.4, J1.5, J3.8, J6.3, J7.2, POWER.5
- new net VCC_8V: R19.2, R20.2, SH1.1, T1.E, T2.C
- new net VDD: IC14.14, IC15.14, IC5.14
- new net VIN: IC4.4, J1.8, J9.PWR, POWER.8, R1.2, T1.C
- new net VSS: IC14.7, IC15.7, IC5.7
- net CLK: now also DIGITAL1.4, J4.4; no longer J1.4, J5.4
- net DIN: now also DIGITAL1.8, J4.8; no longer J1.8, J5.8
- net N$1: now also DIGITAL2.7; no longer J4.7
- net N$17: now also DIGITAL2.2; no longer J4.2
- net N$18: now also J1.1, POWER.1; no longer J2.1, J6.1
- net N$19: now also J1.2, POWER.2; no longer J2.2, J6.2
- net N$20: now also J1.4, POWER.4; no longer J2.4, J6.4
- net N$21: now also IC13.5, R40.2, R41.1; no longer J2.8, J6.8
- net N$22: now also DIGITAL1.6, J4.6; no longer J1.6, J5.6
- net N$31: now also DIGITAL1.3, J4.3; no longer J1.3, J5.3
- net N$34: now also IC8.9, R37.1, R42.2; no longer J1.2, J5.2
- net N$39: now also IC8.8, R37.2, R38.1; no longer J1.1, J5.1
- net N$4: now also DIGITAL1.7, J4.7; no longer J1.7, J5.7
- net N$43: now also DIGITAL2.3; no longer J4.3
- net N$44: now also DIGITAL2.4; no longer J4.4
- net N$45: now also DIGITAL2.5; no longer J4.5
- net N$46: now also DIGITAL2.6; no longer J4.6
- net N$48: now also R43.2, T4.B; no longer J3.8, J4.8
- net N$49: now also DIGITAL2.9; no longer J4.9
- net N$5: now also DIGITAL1.5, J4.5; no longer J1.5, J5.5
- net N$50: now also DIGITAL2.10; no longer J4.10
- net N$52: now also J5.1; no longer JP1.1
- net N$6: now also C8.-, J6.6; no longer ANALOG.4, JP2.4
- net N$7: now also IC13.2, R36.1, R42.1; no longer ANALOG.3, JP2.3
- net N$8: now also J2.5; no longer JP2.5
- net N$9: now also IC13.1, R36.2, R40.1; no longer ANALOG.2, JP2.2
- net RESET: now also C8.+, J1.3, POWER.3; no longer J2.3, J6.3, RESET.3, RESET.4
- net VB: now also DIGITAL2.1; no longer J4.1
Routing:
- net GND: track 9.52 -> 0.00 mm
- net DGND: track 0.00 -> 9.52 mm
- net VCC_5V: track 0.00 -> 7.07 mm
- net RESET: track 50.6 -> 44.0 mm
- net N$48: track 3.90 -> 0.00 mm
- net VIN: track 0.00 -> 3.17 mm
- net N$9: track 3.17 -> 0.00 mm
- net N$7: track 3.17 -> 0.00 mm
- net N$6: track 3.17 -> 0.00 mm
- net N$21: track 3.17 -> 0.00 mm
- net N$122: track 3.17 -> 0.00 mm
- net ADC_RESP: track 0.00 -> 3.17 mm
- net ADC_PPG: track 0.00 -> 3.17 mm
- net ADC_ICG: track 0.00 -> 3.17 mm
- net ADC_ECG: track 0.00 -> 3.17 mm
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- added copper zone on layer 16, net DGND
- removed copper zone on layer 16, net GND

Commit message: Redesign
Parts:
- removed C22: (no value), SparkFun-Capacitors:CAP-PTH-5MM
- removed IC11, IC12, IC13: QUAD_OPAMPP, adafruit:DIL14
- removed IC14, IC15: 4066N, 40xx:DIL14
- removed R28: 100K, adafruit:0204/5
- removed R66: (no value), adafruit:0207/10
- removed R86: (no value), rcl:0207/10
- removed SH1, SH2, SH3: SHORT, stanford_iot_research:R0OHM
- removed T1, T2: 2N2222, adafruit:TO92-EBC-OVAL
- added C17, C18: (no value), SparkFun-Capacitors:CAP-PTH-5MM
- added D2, D4: 5V, diode:ZDIO-2.5
- added D3: 3V, diode:ZDIO-2.5
- added J10: POWER_JACKPTH, SparkFun-Connectors:POWER_JACK_PTH
- added R44: (no value), rcl:0204/5
- added R45, R46, R47, R49, R50: 30K, adafruit:0204/5
- added R48: 50K, adafruit:0204/5
- C9: value 1nF -> (none); device SparkFun-Passives:CAP-PTH-5MM -> SparkFun-Capacitors:CAP-PTH-5MM
- D1: value 5.1V -> 3V; device SparkFun-DiscreteSemi:DIODE-ZENER -> diode:ZDIO-2.5
- IC1, IC3: value LMC660 -> QUAD_OPAMPP
- IC10: value QUAD_OPAMPP -> 4066N; device adafruit:DIL14 -> 40xx:DIL14
- IC5: value 4066N -> QUAD_OPAMPP; device 40xx:DIL14 -> adafruit:DIL14
- IC8: value LMC660 -> LM555N; device adafruit:DIL14 -> linear:DIL08
- IC9: value QUAD_OPAMPP -> LM555N; device adafruit:DIL14 -> linear:DIL08
- R1: value 10K -> (none); device adafruit:0204/5 -> rcl:0204/5
- R11: value 50K -> (none); device adafruit:0204/5 -> rcl:0207/10
- R14: value 30K -> (none); device adafruit:0204/5 -> rcl:0207/10
- R15, R17, R24: value 50K -> 30K
- R16: value 30K -> 50K
- R26: value 16K -> 30K
- R27: value 18K -> 50K
- moved R14 755.6 mm to (-53.3, -817.9)
- moved R19 749.5 mm to (-33.0, -858.5)
- moved R15 724.2 mm to (-35.6, -845.8)
- moved R16 718.6 mm to (-55.9, -858.5)
- moved R17 718.6 mm to (-48.3, -858.5)
- moved C6 717.0 mm to (-33.0, -878.8)
- moved R11 708.0 mm to (-53.3, -812.8)
- moved R22 708.0 mm to (-55.9, -866.1)
- moved C7 706.4 mm to (-55.9, -886.5)
- moved R18 699.8 mm to (-40.6, -858.5)
- moved C1 698.4 mm to (-48.3, -823.0)
- moved R23 689.0 mm to (-48.3, -866.1)
- moved R24 689.0 mm to (-40.6, -866.1)
- moved C5 685.1 mm to (-55.9, -828.0)
- moved R1 661.0 mm to (-55.9, -762.0)
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- renumbered C2 to CE1, C3 to CE3, C4 to CE2, R12 to RE16, R13 to RE17, R2 to RE11, R3 to RE13, R4 to RE12, R5 to RE14, R51 to RE6, R52 to RE4, R53 to RE3, R54 to RE2, R55 to RE9, R56 to RE8, R57 to RE10, R58 to RE5, R6 to RE15, R7 to RE1, R8 to RE7
Connections:
- removed net AGND: C11.1, C12.1, C15.2, C23.2, C32.1, C33.1, C37.2, C38.2, C9.2, CE3.2, IC1.12, IC12.10, IC5.4, IC7.3, J8.10, J8.12, J8.8, R10.1, R100.1, R26.1, R31.1, R33.1, R41.2, R66.2, R68.1, R85.1, R86.1, R9.1, R92.1, R96.1, RE10.2, RE11.1, RE12.1, SH2.2, T3.E, T4.E
- removed net AVCC: IC1.4, R25.2, R29.2, SH1.2
- removed net AVSS: IC1.11, SH3.2
- removed net CLOCK1: C22.1, IC12.1, R83.1, R87.2, R88.2
- removed net DGND: C1.2, C5.2, C6.2, C7.2, D1.P$2, IC2.11, IC4.11, J1.6, J1.7, J6.1, J6.2, J7.3, J9.GND, POWER.6, POWER.7, R11.1, R15.1, R17.1, R21.1, R22.1, R24.1, SH3.1
- removed net N$97: IC12.3, R86.2, R87.1
- removed net V-: IC10.11, IC11.11, IC12.11, IC13.11, IC3.11, IC6.11, IC7.11, IC8.11, IC9.11
- removed net VCC_4V: IC4.6, SH2.1, T2.E
- removed net VCC_8V: R19.2, R20.2, SH1.1, T1.E, T2.C
- removed net VDD: IC14.14, IC15.14, IC5.14
- removed net VIN: IC4.4, J1.8, J9.PWR, POWER.8, R1.2, T1.C
- removed net VSS: IC14.7, IC15.7, IC5.7
- new net +8V: D1.C, IC1.4, IC10.14, IC2.4, IC3.4, IC4.4, IC5.4, IC6.4, IC8.4, IC8.8, IC9.4, IC9.8, J1.8, J9.PWR, POWER.8, R11.2, R20.2, R25.2, R29.2, R87.2
- new net -8V: C1.1, C32.1, C33.2, C5.2, D3.C, IC1.11, IC10.7, IC2.11, IC3.11, IC4.11, IC5.11, IC6.11, IC8.1, IC9.1, J10.GND
- new net 2.5V_BIAS: IC1.6, IC1.7, R16.1, R22.1, R27.1, R48.1
- new net 5V_ADCREF: IC1.1, IC1.2
- new net GND: C11.1, C12.1, C15.2, C18.2, C23.2, C37.2, C38.2, C6.2, C7.2, C9.2, CE3.2, D2.A, D4.A, IC10.4, IC2.12, IC3.12, IC4.5, IC7.11, J1.6, J1.7, J10.PWR, J6.1, J6.2, J7.3, J8.10, J8.12, J8.8, J9.GND, POWER.6, POWER.7, R1.1, R10.1, R100.1, R17.1, R23.1, R31.1, R33.1, R41.2, R44.1, R45.1, R49.1, R68.1, R85.1, R9.1, R92.1, R96.1, RE10.2, RE11.1, RE12.1, T3.E, T4.E
- new net N$54: IC7.2, R17.2, R19.2
- new net N$56: IC7.6, R23.2, R24.2
- new net N$58: C33.1, IC9.5
- new net N$59: IC7.9, R45.2, R46.2
- new net N$60: C18.1, IC7.12, R47.2, R48.2
- new net N$61: IC7.13, R49.2, R50.2
- new net N$63: C17.2, IC9.3
- net 2KHZ_OSC: now also IC10.6; no longer IC14.5, IC6.1, R27.2, R28.2
- net 30KHZ_OSC: now also C17.1, IC10.13, R44.2, R83.1; no longer C22.2, IC5.13, R66.1
- net ADC_ECG: now also IC7.8, R46.1; no longer IC2.8, IC2.9
- net ADC_ICG: now also IC7.1, R19.1; no longer IC2.1, IC2.2
- net ADC_PPG: now also IC7.14, R50.1; no longer IC2.13, IC2.14
- net ADC_RESP: now also IC7.7, R24.1; no longer IC2.6, IC2.7
- net ECG_OUT: now also IC1.13, IC1.14, R26.1; no longer IC1.6, IC1.7, R18.1
- net ICG_DEMUX: now also IC4.1; no longer IC12.14
- net ICG_OUT: now also IC5.1, R15.1; no longer IC11.8, R14.1
- net N$10: now also D1.A, D2.C; no longer IC4.1, T1.B
- net N$100: now also IC5.12; no longer IC12.5
- net N$101: now also IC3.13; no longer IC12.9
- net N$102: now also IC4.3; no longer IC12.12
- net N$103: now also IC5.9; no longer IC11.6
- net N$105: now also IC5.6; no longer IC11.2
- net N$107: now also IC5.8; no longer IC11.7
- net N$108: now also IC5.3; no longer IC11.10
- net N$109: now also IC5.2; no longer IC11.9
- net N$11: now also IC1.10; no longer IC1.3
- net N$12: now also IC1.12; no longer IC1.5
- net N$13: now also IC1.8; no longer IC1.1
- net N$15: now also IC2.14; no longer IC1.14
- net N$16: now also IC2.5; no longer IC9.3
- net N$2: now also IC1.9; no longer IC1.2
- net N$21: now also IC6.10; no longer IC13.5
- net N$23: now also IC3.5; no longer IC10.3
- net N$24: now also IC3.14; no longer IC12.8
- net N$25: now also IC3.6; no longer IC10.2
- net N$26: now also IC2.13; no longer IC1.13
- net N$27: now also IC3.7; no longer IC10.1
- net N$28: now also IC1.3, R20.1, R21.2; no longer C1.1, IC2.3, R14.2, R15.2
- net N$29: now also IC8.7, R14.1; no longer C6.1, IC2.10, R18.2, R22.2
- net N$3: now also IC1.5, R1.2, R21.1; no longer C5.1, IC2.5, R16.2, R17.2
- net N$30: now also C5.1, IC8.5; no longer C7.1, IC2.12, R23.2, R24.2
- net N$32: now also IC9.2, IC9.6, R87.1, R88.2; no longer C33.2, IC12.2, R88.1
- net N$33: now also D3.A, D4.C; no longer IC4.2, R11.2, R19.1
- net N$34: now also IC6.2; no longer IC8.9
- net N$35: now also IC10.1; no longer IC5.1
- net N$36: now also IC9.7, R88.1; no longer D1.P$1, IC4.3, R1.1
- net N$37: now also IC10.2, IC10.3, IC4.2; no longer IC12.13, IC5.2, IC5.3
- net N$38: now also IC8.3, R43.2, T4.B; no longer IC4.5, R20.1, R21.2
- net N$39: now also IC6.1; no longer IC8.8
- net N$40: now also IC5.5; no longer IC11.3
- net N$41: now also C1.2, IC8.2, IC8.6, R11.1, R14.2; no longer IC4.7, T2.B
- net N$42: now also IC6.9; no longer IC13.6
- net N$47: now also IC2.6; no longer IC9.2
- net N$48: now also C6.1, IC7.3, R15.2, R16.2; no longer R43.2, T4.B
- net N$51: now also IC10.5; no longer IC5.5
- net N$53: now also IC6.8; no longer IC13.7
- net N$55: now also C7.1, IC7.5, R18.2, R22.2; no longer C9.1, IC6.2, R28.1
- net N$57: now also C9.1, IC7.10, R27.2; no longer IC6.3, R27.1
- net N$62: now also IC10.11, IC10.8, IC4.7; no longer IC14.4, IC15.4, IC7.1
- net N$64: now also IC4.10; no longer IC7.5
- net N$66: now also IC4.9; no longer IC7.6
- net N$67: now also IC4.8; no longer IC7.7
- net N$69: now also IC2.7; no longer IC9.1
- net N$7: now also IC6.6; no longer IC13.2
- net N$70: now also IC2.10; no longer IC9.5
- net N$71: now also IC2.2; no longer IC1.9
- net N$72: now also IC2.1; no longer IC1.8
- net N$73: now also IC2.3; no longer IC1.10
- net N$74: now also IC3.10; no longer IC10.5
- net N$75: now also IC2.9; no longer IC9.6
- net N$76: now also IC3.2; no longer IC3.9
- net N$77: now also IC2.8; no longer IC9.7
- net N$78: now also IC3.1; no longer IC3.8
- net N$79: now also IC3.3; no longer IC3.10
- net N$80: now also IC3.9; no longer IC10.6
- net N$81: now also IC4.12; no longer IC7.10
- net N$84: now also IC3.8; no longer IC10.7
- net N$9: now also IC6.7; no longer IC13.1
- net N$95: now also IC5.13; no longer IC12.6
- net N$96: now also IC5.10; no longer IC11.5
- net PPG_DP: now also IC4.6; no longer IC7.2
- net PPG_IA_N: now also IC10.10, IC6.5; no longer IC13.3, IC15.3
- net PPG_IA_P: now also IC10.9, IC6.3; no longer IC14.3, IC8.10
- net PPG_LEDN: now also IC10.12; no longer IC15.5
- net PPG_OUT: now also IC4.13, IC4.14, R47.1; no longer IC7.8, IC7.9, R23.1
- net RESP_OUT: now also IC5.7, R18.1; no longer IC11.1, R16.1
- net V+: now also IC5.14; no longer IC10.4, IC11.4, IC12.4, IC12.7, IC13.4, IC3.4, IC6.4, IC7.4, IC8.4, IC9.4
- net VCC_5V: now also IC7.4; no longer IC2.4
Routing:
- net RESET: track 44.0 -> 3.17 mm
- net GND: track 0.00 -> 9.52 mm
- net DGND: track 9.52 -> 0.00 mm
- net VIN: track 3.17 -> 0.00 mm
- net +8V: track 0.00 -> 3.17 mm
Other:
- board size 68.6 x 53.3 mm -> 120.4 x 53.3 mm
- board text removed: "ECG"
- board text removed: "ICG"
- board text removed: "LEVEL SHIFT"
- board text removed: "POWER"

Commit message: Grouped items in layout
Parts:
- removed C20, C21, C23, C24, C29, C32, C33, C34, C35, C36, C37, C38: (no value), SparkFun-Capacitors:CAP-PTH-5MM
- removed R10, R16, R20, R21, R22, R27, R48, R9: 50K, adafruit:0204/5
- removed R100, R11, R14, R87, R88, R91, R99: (no value), rcl:0207/10
- removed R15, R17, R18, R19, R23, R24, R26, R45, R46, R47, R49, R50: 30K, adafruit:0204/5
- removed R25, R69: (no value), resistor:0207/10
- removed R29: 120-320, adafruit:0204/5
- removed R30: 220K, adafruit:0204/5
- removed R31: 160K, adafruit:0204/5
- removed R32: 500K, adafruit:0204/5
- removed R33: 1K-6K, adafruit:0204/5
- removed R34: 2.4K, adafruit:0204/5
- removed R35: 3.9K, adafruit:0204/5
- removed R36, R37: 4.99K, adafruit:0204/5
- removed R38, R39, R40, R41: 9.53K, adafruit:0204/5
- removed R42: (no value), adafruit:0204/5
- removed R43, R61, R62, R63, R64: 10K, adafruit:0204/5
- removed R44: (no value), rcl:0204/5
- removed R59, R60: 24.7K, adafruit:0204/5
- removed R65: 1.3K, adafruit:0204/5
- removed R67, R68, R70, R71, R72, R78, R82, R83, R85, R92, R93, R94, R95, R96, R97, R98: (no value), adafruit:0207/10
- added C19: 1uF, adafruit:E2-5
- added C2, C3, C4: 100uF, SparkFun-Passives:CPOL-RADIAL-100UF-25V
- added CA1, CA2, CA3, CA4, CI1, CI10, CI11, CI12, CI13, CI2, CI3, CI4, CI5, CI6, CI7, CI8, CI9, CP1, CP2: (no value), SparkFun-Capacitors:CAP-PTH-5MM
- added CP3: 22pF, SparkFun-Passives:CAP-PTH-5MM
- added CP4, CP5: 100nF, SparkFun-Passives:CAP-PTH-5MM
- added CP6: 10uF, SparkFun-Passives:CAP-PTH-5MM
- added CP7: 10nF, SparkFun-Passives:CAP-PTH-5MM
- added CP8: 1uF, SparkFun-Passives:CAP-PTH-5MM
- added CP9: 4.3uF, SparkFun-Passives:CAP-PTH-5MM
- added R2, R3, RA10, RA14, RA2, RA6, RI1, RI34: 50K, resistor:0207/10
- added RA1, RA11, RA12, RA13, RA15, RA16, RA3, RA4, RA5, RA7, RA8, RA9: 30K, resistor:0207/10
- added RI10, RI11, RI12, RI13, RI14, RI15, RI16, RI17, RI18, RI19, RI20, RI21, RI22, RI23, RI24, RI25, RI26, RI27, RI28, RI29, RI30, RI31, RI32, RI33, RI9, RP1, RP2, RP9: (no value), resistor:0207/10
- added RI2, RI3, RI7, RI8, RP4: 10K, resistor:0207/10
- added RI4, RI6: 24.7K, resistor:0207/10
- added RI5: 1.3K, resistor:0207/10
- added RP10, RP8: 4.99K, resistor:0207/10
- added RP11, RP12, RP6, RP7: 9.53K, resistor:0207/10
- added RP13: 160K, resistor:0207/10
- added RP14: 1K-6K, resistor:0207/10
- added RP15: 500K, resistor:0207/10
- added RP16: 2.4K, resistor:0207/10
- added RP17: 3.9K, resistor:0207/10
- added RP3: 120-320, resistor:0207/10
- added RP5: 220K, resistor:0207/10
- C1, C17, C18, C5, C6, C7, C9: value (none) -> 100uF; device SparkFun-Capacitors:CAP-PTH-5MM -> SparkFun-Passives:CPOL-RADIAL-100UF-25V
- C10: value 22pF -> 100uF; device SparkFun-Passives:CAP-PTH-5MM -> SparkFun-Passives:CPOL-RADIAL-100UF-25V
- C11, C12: value 100nF -> 100uF; device SparkFun-Passives:CAP-PTH-5MM -> SparkFun-Passives:CPOL-RADIAL-100UF-25V
- C13: value 10uF -> 100uF; device SparkFun-Passives:CAP-PTH-5MM -> SparkFun-Passives:CPOL-RADIAL-100UF-25V
- C14: value 10nF -> 100uF; device SparkFun-Passives:CAP-PTH-5MM -> SparkFun-Passives:CPOL-RADIAL-100UF-25V
- C15: value 1uF -> 100uF; device SparkFun-Passives:CAP-PTH-5MM -> SparkFun-Passives:CPOL-RADIAL-100UF-25V
- C16: value 4.3uF -> 100uF; device SparkFun-Passives:CAP-PTH-5MM -> SparkFun-Passives:CPOL-RADIAL-100UF-25V
- C8: value 1uF -> 100uF; device adafruit:E2-5 -> SparkFun-Passives:CPOL-RADIAL-100UF-25V
- D1, D2, D3, D4: device diode:ZDIO-2.5 -> diode:ZDIO-10
- R1: device rcl:0204/5 -> resistor:0207/10
- RE1, RE10, RE11, RE12, RE13, RE14, RE15, RE16, RE17, RE2, RE3, RE4, RE5, RE6, RE7, RE8, RE9: device adafruit:0204/5 -> resistor:0207/10
- moved C7 976.1 mm to (-17.8, 88.9)
- moved C9 975.5 mm to (-33.0, 88.9)
- moved C6 968.0 mm to (-10.2, 88.9)
- moved C18 950.2 mm to (-17.8, 63.5)
- moved J10 946.9 mm to (78.7, 15.2)
- moved J9 946.9 mm to (78.7, 33.0)
- moved IC7 944.4 mm to (30.5, 92.7)
- moved C1 922.9 mm to (-7.62, 99.1)
- moved C5 918.5 mm to (-2.54, 88.9)
- moved C17 853.7 mm to (-25.4, 63.5)
- moved R1 811.5 mm to (94.0, 35.6)
- moved D1 792.0 mm to (94.0, 30.5)
- moved D2 786.1 mm to (94.0, 25.4)
- moved IC6 784.1 mm to (5.08, -53.3)
- moved D3 780.2 mm to (94.0, 20.3)
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Connections:
- new net RI13: IC10.5, RI22.1, T3.C
- net +8V: now also C1.1, C2.1, C3.1, C4.1, C5.1, C6.1, C7.1, C8.1, C9.1, R3.2, RI14.2, RI22.2, RP2.2, RP3.2; no longer R11.2, R20.2, R25.2, R29.2, R87.2
- net -8V: now also C10.2, C11.2, C12.2, C13.2, C14.2, C15.2, C16.2, C17.2, C18.2, CI4.2, CI5.1, CP1.2, CP2.1; no longer C1.1, C32.1, C33.2, C5.2
- net 2.5V_BIAS: now also RA10.1, RA14.1, RA2.1, RA6.1; no longer R16.1, R22.1, R27.1, R48.1
- net 2KHZ_OSC: now also IC8.3, RP4.1; no longer R43.1
- net 30KHZ_OSC: now also CI6.1, RI13.2, RI16.2, RI20.1; no longer C17.1, R44.2, R83.1, T3.B
- net ADC_ECG: now also RA12.1; no longer R46.1
- net ADC_ICG: now also RA4.1; no longer R19.1
- net ADC_PPG: now also RA16.1; no longer R50.1
- net ADC_RESP: now also RA8.1; no longer R24.1
- net ECG_OUT: now also RA9.1; no longer R26.1
- net ELECTRODE3: now also CI7.1, RI18.2, RI19.1; no longer C29.1, R78.1, R91.2
- net GND: now also C1.2, C10.1, C13.1, C14.1, C15.1, C16.1, C17.1, C18.1, C2.2, C3.2, C4.2, C5.2, C8.2, CA1.2, CA2.2, CA3.2, CA4.2, CI11.2, CI13.2, CI9.2, CP4.1, CP5.1, CP8.2, RA11.1, RA15.1, RA3.1, RA7.1, RI1.1, RI16.1, RI17.1, RI24.1, RI26.1, RI29.1, RI33.1, RI34.1, RP12.2, RP13.1, RP14.1; no longer C15.2, C18.2, C23.2, C37.2, C38.2, R10.1, R100.1, R17.1, R23.1, R31.1, R33.1, R41.2, R44.1, R45.1, R49.1, R68.1, R85.1, R9.1, R92.1, R96.1
- net ICG_DEMUX: now also RI12.2, RI23.1, RI31.1; no longer R67.1, R72.2, R95.1
- net ICG_E1: now also CI1.1; no longer C20.1
- net ICG_E2: now also CI2.1; no longer C21.1
- net ICG_E3: now also CI7.2; no longer C29.2
- net ICG_OUT: now also CI12.2, RA1.1, RI30.2; no longer C36.2, R15.1, R99.2
- net N$100: now also RI17.2, RI18.1; no longer R85.2, R91.1
- net N$101: now also CI3.2, RI9.1; no longer C24.2, R69.1
- net N$102: now also RI10.2, RI12.1; no longer R70.2, R72.1
- net N$103: now also CI10.1, RI25.1, RI26.2; no longer C35.1, R92.2, R93.1
- net N$105: now also RI32.1, RI33.2; no longer R96.2, R97.1
- net N$106: now also CI12.1, RI27.2, RI28.1; no longer C36.1, R94.2, R98.1
- net N$107: now also CI10.2, RI25.2, RI27.1; no longer C35.2, R93.2, R94.1
- net N$108: now also CI11.1, RI28.2; no longer C37.1, R98.2
- net N$109: now also RI29.2, RI30.1; no longer R100.2, R99.1
- net N$110: now also CI8.1, CI9.1, RI23.2; no longer C23.1, C34.1, R67.2
- net N$21: now also RP11.2, RP12.1; no longer R40.2, R41.1
- net N$23: now also CI2.2, RI34.2; no longer C21.2, R10.2
- net N$24: now also CI3.1, RI8.2; no longer C24.1, R64.2
- net N$25: now also RI5.1, RI6.1; no longer R59.1, R65.1
- net N$27: now also RI6.2, RI7.1; no longer R59.2, R63.1
- net N$28: now also R2.2, R3.1; no longer R20.1, R21.2
- net N$29: now also RP1.1; no longer R14.1
- net N$3: now also R2.1; no longer R21.1
- net N$30: now also CP1.1; no longer C5.1
- net N$32: now also CI5.2, RI14.1, RI15.2; no longer C32.2, R87.1, R88.2
- net N$34: now also RP8.1, RP9.2; no longer R37.1, R42.2
- net N$35: now also RI11.2; no longer R71.2
- net N$36: now also RI15.1; no longer R88.1
- net N$38: now also RP4.2; no longer IC8.3, R43.2
- net N$39: now also RP6.1, RP8.2; no longer R37.2, R38.1
- net N$40: now also CI13.1, RI31.2; no longer C38.1, R95.2
- net N$41: now also CP2.2, RP1.2, RP2.1; no longer C1.2, R11.1, R14.2
- net N$42: now also RP6.2, RP7.1; no longer R38.2, R39.1
- net N$48: now also CA1.1, RA1.2, RA2.2; no longer C6.1, R15.2, R16.2
- net N$51: now also RI13.1, T3.B; no longer IC10.5, R25.1, T3.C
- net N$53: now also CP6.1, RP7.2; no longer C13.1, R39.2
- net N$54: now also RA3.2, RA4.2; no longer R17.2, R19.2
- net N$55: now also CA2.1, RA5.2, RA6.2; no longer C7.1, R18.2, R22.2
- net N$56: now also RA7.2, RA8.2; no longer R23.2, R24.2
- net N$57: now also CA3.1, RA10.2, RA9.2; no longer C9.1, R26.2, R27.2
- net N$58: now also CI4.1; no longer C33.1
- net N$59: now also RA11.2, RA12.2; no longer R45.2, R46.2
- net N$6: now also C19.-; no longer C8.-
- net N$60: now also CA4.1, RA13.2, RA14.2; no longer C18.1, R47.2, R48.2
- net N$61: now also RA15.2, RA16.2; no longer R49.2, R50.2
- net N$62: now also CP3.1, RP5.2; no longer C10.1, R30.2
- net N$63: now also CI6.2; no longer C17.2
- net N$64: now also CP6.2, RP13.2; no longer C13.2, R31.2
- net N$66: now also CP7.2, RP14.2, RP15.1; no longer C14.2, R32.1, R33.2
- net N$67: now also CP7.1, RP15.2, RP16.1; no longer C14.1, R32.2, R34.1
- net N$68: now also CP9.1, RP16.2, RP17.1; no longer C16.1, R34.2, R35.1
- net N$7: now also RP10.1, RP9.1; no longer R36.1, R42.1
- net N$74: now also RI7.2, RI8.1; no longer R63.2, R64.1
- net N$76: now also RI4.1, RI5.2; no longer R60.1, R65.2
- net N$78: now also RI2.1, RI4.2; no longer R60.2, R61.1
- net N$79: now also CI1.2, RI1.2; no longer C20.2, R9.2
- net N$80: now also RI2.2, RI3.1; no longer R61.2, R62.1
- net N$81: now also CP8.1, RP17.2; no longer C15.1, R35.2
- net N$84: now also RI10.1, RI11.1, RI3.2, RI9.2; no longer R62.2, R69.2, R70.1, R71.1
- net N$9: now also RP10.2, RP11.1; no longer R36.2, R40.1
- net N$95: now also RI20.2, RI21.1; no longer R82.1, R83.2
- net N$96: now also CI8.2, RI24.2; no longer C34.2, R68.2
- net PPG_DP: now also CP3.2, RP5.1; no longer C10.2, R30.1
- net PPG_IA_N: now also CP5.2; no longer C11.2
- net PPG_IA_P: now also CP4.2; no longer C12.2
- net PPG_LEDP: now also RP3.1; no longer R29.1
- net PPG_OUT: now also CP9.2, RA13.1; no longer C16.2, R47.1
- net RESET: now also C19.+; no longer C8.+
- net RESP_OUT: now also RA5.1, RI32.2; no longer R18.1, R97.2
- net V+: now also RI19.2, RI21.2; no longer R78.2, R82.2

Commit message: ICG somewhat good
Parts:
- moved J8 257.6 mm to (-176.5, 3.81), turned to 270 degrees
- moved C3 164.5 mm to (-143.5, -12.7), turned to 90 degrees
- moved C4 149.4 mm to (-148.6, 7.62)
- moved RI34 142.6 mm to (-171.4, 16.5), turned to 180 degrees
- moved C11 133.5 mm to (-138.4, 7.62)
- moved C2 129.4 mm to (-110.5, 11.4)
- moved C10 124.4 mm to (-146.1, 26.7), turned to 180 degrees
- moved C5 110.6 mm to (-85.1, 15.2)
- moved C1 108.7 mm to (-85.1, 22.9)
- moved IC9 108.3 mm to (-109.2, 20.3), turned to 180 degrees
- moved RI18 106.8 mm to (-163.8, 6.35), turned to 270 degrees
- moved RI17 106.3 mm to (-166.4, 6.35), turned to 90 degrees
- moved IC5 104.7 mm to (-143.5, -2.54)
- moved RI19 104.2 mm to (-161.3, 6.35), turned to 90 degrees
- moved RI20 102.6 mm to (-158.8, 6.35), turned to 270 degrees
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Routing:
- net GND: track 9.52 -> 264.3 mm, vias 0 -> 5
- net +8V: track 3.17 -> 190.3 mm, vias 0 -> 8
- net -8V: track 0.00 -> 172.7 mm, vias 0 -> 4
- net 30KHZ_OSC: track 0.00 -> 138.3 mm, vias 0 -> 4
- net N$84: track 0.00 -> 110.0 mm, vias 0 -> 5
- net ICG_DEMUX: track 0.00 -> 67.4 mm, vias 0 -> 4
- net ICG_OUT: track 0.00 -> 55.4 mm, vias 0 -> 2
- net N$103: track 0.00 -> 47.4 mm, vias 0 -> 1
- net N$40: track 0.00 -> 47.3 mm, vias 0 -> 1
- net N$105: track 0.00 -> 45.3 mm, vias 0 -> 5
- net N$27: track 0.00 -> 43.8 mm, vias 0 -> 2
- net N$108: track 0.00 -> 38.4 mm, vias 0 -> 2
- net N$80: track 0.00 -> 38.3 mm
- net N$23: track 0.00 -> 37.7 mm
- net N$109: track 0.00 -> 37.7 mm
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Other:
- board size 120.4 x 53.3 mm -> 60.7 x 53.3 mm
