File: bioshield.brd (EAGLE design)
At the start: 60.7 x 53.3 mm, 165 parts, among them IC1 QUAD_OPAMPP, IC10 4066N, IC2 QUAD_OPAMPP, IC3 QUAD_OPAMPP, IC4 QUAD_OPAMPP, IC5 QUAD_OPAMPP, IC6 QUAD_OPAMPP, IC7 QUAD_OPAMPP, IC8 LM555N, IC9 LM555N, J10 POWER_JACKPTH, J6 FTDI/EZ-LINK, J7 HC-05/HC-06, J8 ELECTRODES, J9 POWER_JACKPTH, T3 2N2222, T4 2N2222

Commit message: Revision 1
Parts:
- removed C14, C6, C9: 100uF, SparkFun-Passives:CPOL-RADIAL-100UF-25V
- removed DIGITAL2: (no value), SmartPrj:1X10-TH
- removed J2: (no value), pinhead:1X05
- removed J4, POWER: (no value), SmartPrj:1X08-TH
- removed J5: (no value), pinhead:1X01
- added R4: 100, resistor:0207/10
- added RP18: 10K, resistor:0207/10
- moved RE12 184.5 mm to (69.8, -5.08), turned to 270 degrees
- moved J8 184.2 mm to (7.62, 1.27), turned to 90 degrees
- moved RE13 182.1 mm to (64.8, -14.0), turned to 180 degrees
- moved CI1 173.6 mm to (-3.81, -12.7), turned to 180 degrees
- moved CI2 171.2 mm to (-3.81, -5.08), turned to 180 degrees
- moved RE6 169.2 mm to (40.6, -5.08), turned to 90 degrees
- moved RE14 168.7 mm to (52.1, -14.0), turned to 180 degrees
- moved RI1 167.7 mm to (-6.35, -10.2), turned to 0 degrees
- moved RE15 167.6 mm to (63.5, 3.81)
- moved RI34 166.9 mm to (-6.35, -7.62), turned to 0 degrees
- moved RE8 165.6 mm to (43.2, -5.08), turned to 270 degrees
- moved CE2 163.9 mm to (52.1, -16.5)
- moved RE5 163.8 mm to (34.3, -14.0), turned to 180 degrees
- moved RE11 159.9 mm to (43.2, 3.81)
- moved RE16 159.9 mm to (34.3, -16.5)
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Connections:
- net PPG_IA_N renamed PPG_IAN
- net PPG_IA_P renamed PPG_IAP
- removed net CLK: DIGITAL1.4, J4.4
- removed net DIN: DIGITAL1.8, J4.8
- removed net N$1: DIGITAL2.7, J3.7
- removed net N$17: DIGITAL2.2, J3.2
- removed net N$18: J1.1, POWER.1
- removed net N$19: J1.2, POWER.2
- removed net N$20: J1.4, POWER.4
- removed net N$22: DIGITAL1.6, J4.6
- removed net N$31: DIGITAL1.3, J4.3
- removed net N$4: DIGITAL1.7, J4.7
- removed net N$43: DIGITAL2.3, J3.3
- removed net N$44: DIGITAL2.4, J3.4
- removed net N$45: DIGITAL2.5, J3.5
- removed net N$46: DIGITAL2.6, J3.6
- removed net N$49: DIGITAL2.9, J3.9
- removed net N$5: DIGITAL1.5, J4.5
- removed net N$50: DIGITAL2.10, J3.10
- removed net N$52: ANALOG.6, J5.1
- removed net N$8: ANALOG.5, J2.5
- removed net VB: DIGITAL2.1, J3.1
- new net N$10000: IC8.3, RP4.1
- new net N$65: IC10.12, R4.2
- net +8V: no longer C6.1, C9.1, POWER.8
- net -8V: no longer C14.2
- net 2KHZ_OSC: now also RP18.2, RP4.2, T4.B; no longer IC10.6, IC8.3, RP4.1
- net 5V_ADCREF: now also J3.8
- net ADC_ECG: no longer J2.2
- net ADC_ICG: no longer J2.4
- net ADC_PPG: no longer J2.1
- net ADC_RESP: no longer J2.3
- net GND: no longer C14.1, C6.2, C9.2, POWER.6, POWER.7
- net N$38: now also IC10.6, RP18.1; no longer RP4.2, T4.B
- net PPG_LEDN: now also R4.1; no longer IC10.12
- net RESET: no longer POWER.3
- net RX: no longer J4.1
- net TX: no longer J4.2
- net VCC_5V: no longer DIGITAL2.8, J3.8, POWER.5
Routing:
- net +8V: track 190.3 -> 499.9 mm, vias 8 -> 15
- net -8V: track 172.7 -> 477.9 mm, vias 4 -> 6
- net 5V_ADCREF: track 0.00 -> 135.6 mm
- net RESP_OUT: track 29.7 -> 140.7 mm, vias 2 -> 3
- net 2.5V_BIAS: track 0.00 -> 106.5 mm
- net RX: track 3.17 -> 86.4 mm
- net ICG_OUT: track 55.4 -> 132.6 mm, vias 2 -> 1
- net TX: track 3.17 -> 79.3 mm
- net N$28: track 0.00 -> 64.1 mm
- net N$3: track 0.00 -> 62.7 mm
- net N$58: track 8.69 -> 70.8 mm
- net N$16: track 0.00 -> 61.6 mm
- net PPG_DP: track 0.00 -> 59.6 mm, vias 0 -> 1
- net ECG_OUT: track 0.00 -> 59.5 mm
- net ADC_PPG: track 3.17 -> 62.1 mm
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- added copper zone on layer 1, net GND
- added copper zone on layer 16, net GND
- removed copper zone on layer 16, net DGND
Other:
- board size 60.7 x 53.3 mm -> 138.4 x 81.3 mm
- board text added: "EE122B Bioshield v1"
- board text removed: "3.3V"
- board text removed: "ANALOG"
- board text removed: "RST"
- board text removed: "VIN"
