File: bioshield.brd (EAGLE design)
At the start: 138.4 x 81.3 mm, 159 parts, among them IC1 QUAD_OPAMPP, IC10 4066N, IC2 QUAD_OPAMPP, IC3 QUAD_OPAMPP, IC4 QUAD_OPAMPP, IC5 QUAD_OPAMPP, IC6 QUAD_OPAMPP, IC7 QUAD_OPAMPP, IC8 LM555N, IC9 LM555N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

Commit message: Pre-assembly
Parts:
- R1: value (none) -> 25K
- R2, RA10, RA14, RA2, RA6: value 50K -> 25K
- R3: value 50K -> 30K
- RA1, RA11, RA13, RA15, RA3, RA5, RA7, RA9: value 30K -> 80K
- RA12, RA16, RA4, RA8: value 30K -> 25K
Changed lines of the file:
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@@
 <attribute name="NAME" x="-25.019" y="14.478" size="1" layer="25" font="vector" ratio="10" rot="R270"/>
 </element>
-<element name="R3" library="resistor" package="0207/10" value="50K" x="58.42" y="45.72" smashed="yes">
+<element name="R3" library="resistor" package="0207/10" value="30K" x="58.42" y="45.72" smashed="yes">
 <attribute name="NAME" x="65.024" y="45.466" size="1" layer="25" font="vector" ratio="10"/>
 </element>
-<element name="R2" library="resistor" package="0207/10" value="50K" x="58.42" y="50.8" smashed="yes" rot="R180">
+<element name="R2" library="resistor" package="0207/10" value="25K" x="58.42" y="50.8" smashed="yes" rot="R180">
 <attribute name="NAME" x="66.548" y="51.562" size="1" layer="25" font="vector" ratio="10" rot="R180"/>
 </element>
@@
 <attribute name="NAME" x="56.0832" y="35.4838" size="1" layer="25" font="vector" ratio="10" rot="R90"/>
 </element>
-<element name="R1" library="resistor" package="0207/10" value="" x="58.42" y="48.26" smashed="yes">
+<element name="R1" library="resistor" package="0207/10" value="25K" x="58.42" y="48.26" smashed="yes">
 <attribute name="NAME" x="65.024" y="48.006" size="1" layer="25" font="vector" ratio="10"/>
 <attribute name="VALUE" x="56.1594" y="47.625" size="1.27" layer="27" ratio="10"/>
@@
 <attribute name="NAME" x="9.398" y="25.019" size="1" layer="25" font="vector" ratio="10" rot="R180"/>
 </element>
-<element name="RA1" library="resistor" package="0207/10" value="30K" x="31.75" y="50.8" smashed="yes">
+<element name="RA1" library="resistor" package="0207/10" value="80K" x="31.75" y="50.8" smashed="yes">
 <attribute name="NAME" x="28.702" y="52.324" size="1" layer="25" font="vector" ratio="10"/>
 </element>
-<element name="RA2" library="resistor" package="0207/10" value="50K" x="38.1" y="22.86" smashed="yes" rot="R180">
+<element name="RA2" library="resistor" package="0207/10" value="25K" x="38.1" y="22.86" smashed="yes" rot="R180">
 <attribute name="NAME" x="41.148" y="21.336" size="1" layer="25" font="vector" ratio="10" rot="R180"/>
 </element>
@@
 <attribute name="NAME" x="18.669" y="27.432" size="1" layer="25" font="vector" ratio="10" rot="R90"/>
 </element>
-<element name="RA3" library="resistor" package="0207/10" value="30K" x="25.4" y="22.86" smashed="yes" rot="R180">
+<element name="RA3" library="resistor" package="0207/10" value="80K" x="25.4" y="22.86" smashed="yes" rot="R180">
 <attribute name="NAME" x="28.448" y="21.336" size="1" layer="25" font="vector" ratio="10" rot="R180"/>
 </element>
-<element name="RA4" library="resistor" package="0207/10" value="30K" x="38.1" y="20.32" smashed="yes">
+<element name="RA4" library="resistor" package="0207/10" value="25K" x="38.1" y="20.32" smashed="yes">
 <attribute name="NAME" x="35.052" y="21.844" size="1" layer="25" font="vector" ratio="10"/>
 </element>
-<element name="RA5" library="resistor" package="0207/10" value="30K" x="38.1" y="17.78" smashed="yes" rot="R180">
+<element name="RA5" library="resistor" package="0207/10" value="80K" x="38.1" y="17.78" smashed="yes" rot="R180">
 <attribute name="NAME" x="41.148" y="16.256" size="1" layer="25" font="vector" ratio="10" rot="R180"/>
 </element>
-<element name="RA6" library="resistor" package="0207/10" value="50K" x="38.1" y="15.24" smashed="yes" rot="R180">
+<element name="RA6" library="resistor" package="0207/10" value="25K" x="38.1" y="15.24" smashed="yes" rot="R180">
 <attribute name="NAME" x="41.148" y="13.716" size="1" layer="25" font="vector" ratio="10" rot="R180"/>
 </element>
@@
 <attribute name="VALUE" x="35.306" y="42.926" size="0.4064" layer="27" rot="R270"/>
 </element>
-<element name="RA7" library="resistor" package="0207/10" value="30K" x="25.4" y="17.78" smashed="yes" rot="R180">
+<element name="RA7" library="resistor" package="0207/10" value="80K" x="25.4" y="17.78" smashed="yes" rot="R180">
 <attribute name="NAME" x="28.448" y="16.256" size="1" layer="25" font="vector" ratio="10" rot="R180"/>
 </element>
-<element name="RA8" library="resistor" package="0207/10" value="30K" x="25.4" y="20.32" smashed="yes" rot="R180">
+<element name="RA8" library="resistor" package="0207/10" value="25K" x="25.4" y="20.32" smashed="yes" rot="R180">
 <attribute name="NAME" x="28.448" y="18.796" size="1" layer="25" font="vector" ratio="10" rot="R180"/>
 </element>
-<element name="RA9" library="resistor" package="0207/10" value="30K" x="49.53" y="29.21" smashed="yes" rot="R270">
+<element name="RA9" library="resistor" package="0207/10" value="80K" x="49.53" y="29.21" smashed="yes" rot="R270">
 <attribute name="NAME" x="49.276" y="30.734" size="1" layer="25" font="vector" ratio="10" rot="R270"/>
 </element>
-<element name="RA10" library="resistor" package="0207/10" value="50K" x="45.72" y="29.21" smashed="yes" rot="R270">
+<element name="RA10" library="resistor" package="0207/10" value="25K" x="45.72" y="29.21" smashed="yes" rot="R270">
 <attribute name="NAME" x="45.212" y="31.242" size="1" layer="25" font="vector" ratio="10" rot="R270"/>
 </element>
@@
 <attribute name="VALUE" x="41.656" y="30.226" size="0.4064" layer="27" rot="R270"/>
 </element>
-<element name="RA11" library="resistor" package="0207/10" value="30K" x="45.72" y="44.45" smashed="yes">
+<element name="RA11" library="resistor" package="0207/10" value="80K" x="45.72" y="44.45" smashed="yes">
 <attribute name="NAME" x="42.672" y="45.974" size="1" layer="25" font="vector" ratio="10"/>
 </element>
-<element name="RA12" library="resistor" package="0207/10" value="30K" x="45.72" y="41.91" smashed="yes" rot="R180">
+<element name="RA12" library="resistor" package="0207/10" value="25K" x="45.72" y="41.91" smashed="yes" rot="R180">
 <attribute name="NAME" x="48.514" y="40.132" size="1" layer="25" font="vector" ratio="10" rot="R180"/>
 </element>
-<element name="RA13" library="resistor" package="0207/10" value="30K" x="25.4" y="39.37" smashed="yes">
+<element name="RA13" library="resistor" package="0207/10" value="80K" x="25.4" y="39.37" smashed="yes">
 <attribute name="NAME" x="22.352" y="40.894" size="1" layer="25" font="vector" ratio="10"/>
 </element>
-<element name="RA14" library="resistor" package="0207/10" value="50K" x="25.4" y="41.91" smashed="yes">
+<element name="RA14" library="resistor" package="0207/10" value="25K" x="25.4" y="41.91" smashed="yes">
 <attribute name="NAME" x="22.352" y="43.434" size="1" layer="25" font="vector" ratio="10"/>
 </element>
@@
 <attribute name="VALUE" x="39.116" y="30.226" size="0.4064" layer="27" rot="R270"/>
 </element>
-<element name="RA15" library="resistor" package="0207/10" value="30K" x="31.75" y="48.26" smashed="yes" rot="R180">
+<element name="RA15" library="resistor" package="0207/10" value="80K" x="31.75" y="48.26" smashed="yes" rot="R180">
 <attribute name="NAME" x="34.798" y="46.736" size="1" layer="25" font="vector" ratio="10" rot="R180"/>
 </element>
-<element name="RA16" library="resistor" package="0207/10" value="30K" x="25.4" y="44.45" smashed="yes" rot="R180">
+<element name="RA16" library="resistor" package="0207/10" value="25K" x="25.4" y="44.45" smashed="yes" rot="R180">
 <attribute name="NAME" x="28.448" y="42.926" size="1" layer="25" font="vector" ratio="10" rot="R180"/>
 </element>
@@
 </signal>
 </signals>
-<errors>
-</errors>
 </board>
 </drawing>
