File: bioshield.sch (EAGLE design)
At the start: 10 parts

Commit message: Schematic nearly complete
Parts:
- removed JP1: (no value), pinhead:PINHD-1X1
- removed JP2: (no value), pinhead:PINHD-1X5
- removed RESET: (no value), switch-omron:10-XX
- added C1, C20, C21, C22, C23, C24, C29, C32, C33, C34, C35, C36, C37, C38, C5, C6, C7: (no value), SparkFun-Capacitors:CAPPTH1
- added C10: 22pF, SparkFun-Passives:CAPPTH1
- added C11, C12, C3: 100nF, SparkFun-Passives:CAPPTH1
- added C13: 10uF, SparkFun-Passives:CAPPTH1
- added C14: 10nF, SparkFun-Passives:CAPPTH1
- added C15: 1uF, SparkFun-Passives:CAPPTH1
- added C16: 4.3uF, SparkFun-Passives:CAPPTH1
- added C2: 3.2u, SparkFun-Passives:CAPPTH1
- added C4: 220nF, SparkFun-Passives:CAPPTH1
- added C8: 1uF, adafruit:CPOL-USE2-5
- added C9: 1nF, SparkFun-Passives:CAPPTH1
- added D1: 5.1V, SparkFun-DiscreteSemi:DIODE-ZENERPTH
- added DIGITAL1, POWER: (no value), SmartPrj:PINHD-1X8TH
- added DIGITAL2: (no value), SmartPrj:PINHD-1X10TH
- added IC1, IC3, IC8: LMC660, adafruit:QUAD_OPAMPP
- added IC10, IC11, IC12, IC13, IC2, IC4, IC6, IC7, IC9: QUAD_OPAMPP, adafruit:QUAD_OPAMPP
- added IC14, IC15, IC5: 4066N, 40xx:4066N
- added J7: HC-05/HC-06, pinhead:PINHD-1X6
- added J8: ELECTRODES, SparkFun-Connectors:M06X2PTH_FEMALE
- added J9: POWER_JACKPTH, SparkFun-Connectors:POWER_JACKPTH
- added R1, R4, R43, R54, R55, R56, R57, R6, R61, R62, R63, R64: 10K, adafruit:R-US_0204/5
- added R10, R11, R15, R17, R20, R21, R22, R24, R7, R8, R9: 50K, adafruit:R-US_0204/5
- added R100, R86, R87, R88, R91, R99: (no value), rcl:R-US_0207/10
- added R12, R2: 1M, adafruit:R-US_0204/5
- added R13: 5M, adafruit:R-US_0204/5
- added R14, R16, R18, R19, R23: 30K, adafruit:R-US_0204/5
- added R25, R69: (no value), resistor:R-US_0207/10
- added R26: 16K, adafruit:R-US_0204/5
- added R27: 18K, adafruit:R-US_0204/5
- added R28: 100K, adafruit:R-US_0204/5
- added R29: 120-320, adafruit:R-US_0204/5
- added R3: 40K, adafruit:R-US_0204/5
- added R30: 220K, adafruit:R-US_0204/5
- added R31: 160K, adafruit:R-US_0204/5
- added R32: 500K, adafruit:R-US_0204/5
- added R33: 1K-6K, adafruit:R-US_0204/5
- added R34: 2.4K, adafruit:R-US_0204/5
- added R35: 3.9K, adafruit:R-US_0204/5
- added R36, R37: 4.99K, adafruit:R-US_0204/5
- added R38, R39, R40, R41: 9.53K, adafruit:R-US_0204/5
- added R42: (no value), adafruit:R-US_0204/5
- added R5: 5.1K, adafruit:R-US_0204/5
- added R51, R52, R59, R60: 24.7K, adafruit:R-US_0204/5
- added R53, R58, R65: 1.3K, adafruit:R-US_0204/5
- added R66, R67, R68, R70, R71, R72, R78, R82, R83, R85, R92, R93, R94, R95, R96, R97, R98: (no value), adafruit:R-US_0207/10
- added SH1, SH2, SH3: SHORT, stanford_iot_research:SHORT
- added T1, T2, T3, T4: 2N2222, adafruit:2N2222
- J2: device SmartPrj:PINHD-1X8TH -> pinhead:PINHD-1X5
- J4: device SmartPrj:PINHD-1X10TH -> SmartPrj:PINHD-1X8TH
- J5: device SmartPrj:PINHD-1X8TH -> pinhead:PINHD-1X1
- J6: value (none) -> FTDI/EZ-LINK; device SmartPrj:PINHD-1X8TH -> pinhead:PINHD-1X6
Connections:
- removed net +5V: J2.5, J6.5
- removed net GND: J2.6, J2.7, J6.6, J6.7, RESET.S, RESET.S1
- removed net N$122: ANALOG.1, JP2.1
- new net 2KHZ_OSC: IC14B.C, IC6A.OUT, R27.2, R28.2, R43.1
- new net 30KHZ_OSC: C22.2, IC5A.C, R66.1, T3.B
- new net ADC_ECG: ANALOG.2, IC2C.-IN, IC2C.OUT, J2.2
- new net ADC_ICG: ANALOG.4, IC2A.-IN, IC2A.OUT, J2.4
- new net ADC_PPG: ANALOG.1, IC2D.-IN, IC2D.OUT, J2.1
- new net ADC_RESP: ANALOG.3, IC2B.-IN, IC2B.OUT, J2.3
- new net AGND: C11.1, C12.1, C15.2, C23.2, C3.2, C32.1, C33.1, C37.2, C38.2, C9.2, IC12C.+IN, IC1D.+IN, IC5B.A, IC7A.+IN, J8.10, J8.12, J8.8, R10.1, R100.1, R2.1, R26.1, R31.1, R33.1, R4.1, R41.2, R57.2, R66.2, R68.1, R85.1, R86.1, R9.1, R92.1, R96.1, SH2.2, T3.E, T4.E
- new net AVCC: IC1P.V+, R25.2, R29.2, SH1.2
- new net AVSS: IC1P.V-, SH3.2
- new net CLOCK1: C22.1, IC12A.OUT, R83.1, R87.2, R88.2
- new net DGND: C1.2, C5.2, C6.2, C7.2, D1.A, IC2P.V-, IC4P.V-, J1.6, J1.7, J6.1, J6.2, J7.3, J9.GND, POWER.6, POWER.7, R11.1, R15.1, R17.1, R21.1, R22.1, R24.1, SH3.1
- new net ECG_E1: J8.1, R7.1
- new net ECG_E2: J8.3, R8.1
- new net ECG_E3: J8.5, R12.2, R13.2
- new net ECG_OUT: C4.2, IC1B.-IN, IC1B.OUT, R18.1
- new net ELECTRODE3: C29.1, R78.1, R91.2
- new net ICG_DEMUX: IC12D.OUT, R67.1, R72.2, R95.1
- new net ICG_E1: C20.1, J8.7
- new net ICG_E2: C21.1, J8.9
- new net ICG_E3: C29.2, J8.11
- new net ICG_OUT: C36.2, IC11C.OUT, R14.1, R99.2
- new net N$10: IC4A.OUT, T1.B
- new net N$100: IC12B.+IN, R85.2, R91.1
- new net N$101: C24.2, IC12C.-IN, R69.1
- new net N$102: IC12D.+IN, R70.2, R72.1
- new net N$103: C35.1, IC11B.-IN, R92.2, R93.1
- new net N$105: IC11A.-IN, R96.2, R97.1
- new net N$106: C36.1, R94.2, R98.1
- new net N$107: C35.2, IC11B.OUT, R93.2, R94.1
- new net N$108: C37.1, IC11C.+IN, R98.2
- new net N$109: IC11C.-IN, R100.2, R99.1
- new net N$11: C2.2, IC1A.+IN, R2.2
- new net N$110: C23.1, C34.1, R67.2
- new net N$12: C3.1, IC1B.+IN, R6.2
- new net N$13: IC1A.OUT, R3.2, R5.1
- new net N$14: C4.1, R5.2, R6.1
- new net N$15: IC1D.OUT, R13.1
- new net N$16: IC9A.+IN, R8.2
- new net N$2: IC1A.-IN, R3.1, R4.2
- new net N$23: C21.2, IC10A.+IN, R10.2
- new net N$24: C24.1, IC12C.OUT, R64.2
- new net N$25: IC10A.-IN, R59.1, R65.1
- new net N$26: IC1D.-IN, R12.1, R53.1, R58.2
- new net N$27: IC10A.OUT, R59.2, R63.1
- new net N$28: C1.1, IC2A.+IN, R14.2, R15.2
- new net N$29: C6.1, IC2C.+IN, R18.2, R22.2
- new net N$3: C5.1, IC2B.+IN, R16.2, R17.2
- new net N$30: C7.1, IC2D.+IN, R23.2, R24.2
- new net N$32: C32.2, C33.2, IC12A.-IN, R88.1
- new net N$33: IC4A.-IN, R11.2, R19.1
- new net N$35: IC5A.A, R71.2
- new net N$36: D1.C, IC4A.+IN, R1.1
- new net N$37: IC12D.-IN, IC5A.B, IC5B.B
- new net N$38: IC4B.+IN, R20.1, R21.2
- new net N$40: C38.1, IC11A.+IN, R95.2
- new net N$41: IC4B.OUT, T2.B
- new net N$42: IC13B.-IN, R38.2, R39.1
- new net N$47: IC9A.-IN, R51.1, R58.1
- new net N$51: IC5B.C, R25.1, T3.C
- new net N$53: C13.1, IC13B.OUT, R39.2
- new net N$55: C9.1, IC6A.-IN, R28.1
- new net N$57: IC6A.+IN, R26.2, R27.1
- new net N$62: C10.1, IC14B.A, IC15B.A, IC7A.OUT, R30.2
- new net N$64: C13.2, IC7B.+IN, R31.2
- new net N$66: C14.2, IC7B.-IN, R32.1, R33.2
- new net N$67: C14.1, IC7B.OUT, R32.2, R34.1
- new net N$68: C16.1, R34.2, R35.1
- new net N$69: IC9A.OUT, R51.2, R56.1
- new net N$70: IC9B.+IN, R56.2, R57.1
- new net N$71: IC1C.-IN, R52.1, R53.2
- new net N$72: IC1C.OUT, R52.2, R54.1
- new net N$73: IC1C.+IN, R7.2
- new net N$74: IC10B.+IN, R63.2, R64.1
- new net N$75: IC9B.-IN, R54.2, R55.1
- new net N$76: IC3C.-IN, R60.1, R65.2
- new net N$77: C2.1, IC9B.OUT, R55.2
- new net N$78: IC3C.OUT, R60.2, R61.1
- new net N$79: C20.2, IC3C.+IN, R9.2
- new net N$80: IC10B.-IN, R61.2, R62.1
- new net N$81: C15.1, IC7C.+IN, R35.2
- new net N$84: IC10B.OUT, R62.2, R69.2, R70.1, R71.1
- new net N$95: IC12B.-IN, R82.1, R83.2
- new net N$96: C34.2, IC11B.+IN, R68.2
- new net N$97: IC12A.+IN, R86.2, R87.1
- new net PPG_DP: C10.2, IC7A.-IN, J8.6, R30.1
- new net PPG_IA_N: C11.2, IC13A.+IN, IC15B.B
- new net PPG_IA_P: C12.2, IC14B.B, IC8C.+IN
- new net PPG_LEDN: IC15B.C, J8.4, T4.C
- new net PPG_LEDP: J8.2, R29.1
- new net PPG_OUT: C16.2, IC7C.-IN, IC7C.OUT, R23.1
- new net RESP_OUT: IC11A.OUT, R16.1, R97.2
- new net RX: DIGITAL1.1, J4.1, J6.4, J7.4
- new net TX: DIGITAL1.2, J4.2, J6.5, J7.5
- new net V+: IC12B.OUT, R78.2, R82.2
- new net VCC_4V: IC4B.-IN, SH2.1, T2.E
- new net VCC_5V: DIGITAL2.8, IC2P.V+, J1.5, J3.8, J6.3, J7.2, POWER.5
- new net VCC_8V: R19.2, R20.2, SH1.1, T1.E, T2.C
- new net VIN: IC4P.V+, J1.8, J9.PWR, POWER.8, R1.2, T1.C
- net CLK: now also DIGITAL1.4, J4.4; no longer J1.4, J5.4
- net DIN: now also DIGITAL1.8, J4.8; no longer J1.8, J5.8
- net N$1: now also DIGITAL2.7; no longer J4.7
- net N$17: now also DIGITAL2.2; no longer J4.2
- net N$18: now also J1.1, POWER.1; no longer J2.1, J6.1
- net N$19: now also J1.2, POWER.2; no longer J2.2, J6.2
- net N$20: now also J1.4, POWER.4; no longer J2.4, J6.4
- net N$21: now also IC13B.+IN, R40.2, R41.1; no longer J2.8, J6.8
- net N$22: now also DIGITAL1.6, J4.6; no longer J1.6, J5.6
- net N$31: now also DIGITAL1.3, J4.3; no longer J1.3, J5.3
- net N$34: now also IC8C.-IN, R37.1, R42.2; no longer J1.2, J5.2
- net N$39: now also IC8C.OUT, R37.2, R38.1; no longer J1.1, J5.1
- net N$4: now also DIGITAL1.7, J4.7; no longer J1.7, J5.7
- net N$43: now also DIGITAL2.3; no longer J4.3
- net N$44: now also DIGITAL2.4; no longer J4.4
- net N$45: now also DIGITAL2.5; no longer J4.5
- net N$46: now also DIGITAL2.6; no longer J4.6
- net N$48: now also R43.2, T4.B; no longer J3.8, J4.8
- net N$49: now also DIGITAL2.9; no longer J4.9
- net N$5: now also DIGITAL1.5, J4.5; no longer J1.5, J5.5
- net N$50: now also DIGITAL2.10; no longer J4.10
- net N$52: now also J5.1; no longer JP1.1
- net N$6: now also C8.-, J6.6; no longer ANALOG.4, JP2.4
- net N$7: now also IC13A.-IN, R36.1, R42.1; no longer ANALOG.3, JP2.3
- net N$8: now also J2.5; no longer JP2.5
- net N$9: now also IC13A.OUT, R36.2, R40.1; no longer ANALOG.2, JP2.2
- net RESET: now also C8.+, J1.3, POWER.3; no longer J2.3, J6.3, RESET.P, RESET.P1
- net VB: now also DIGITAL2.1; no longer J4.1
Other:
- note added: "(PPG_DN)"
- note added: "(PPG_GND)"
- note added: "0/RX"
- note added: "1/TX"
- note added: "10/PWM"
- note added: "11/PWM"
- note added: "12"
- note added: "13"
- note added: "2"
- note added: "2kHz Oscillator"
- note added: "3/PWM"
- note added: "30KHz Oscillator"
- note added: "3V3"
- note added: "4"
- note added: "5/PWM"
- note added: "5V"
- note added: "6/PWM"
- note added: "7"
- note added: "8"
- note added: "8V Regulator"
- note added: "9/PWM"
- note added: "A0"
- note added: "A1"
- note added: "A2"
- note added: "A3"
- note added: "A4"
- note added: "A5"
- note added: "AC Coupling"
- note added: "ADC INPUT"
- note added: "AGND is NOT DGND\!\!"
- note added: "AREF"
- note added: "Arduino Headers"
- note added: "Arduino-compatible headers are provided, with all signals passed through. This allows for stacking additional shields or using alternate Arduino-compatible processors. Power is provided EITHER through the DC power jack OR directly into the VIN pin. They are shorted together, so do not connect multiple power supplies to this pin\! Two standard serial->Bluetooth headers are broken out. J6 is compat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"
- note added: "BIOSHIELD INTERFACE"
- note added: "BPF"
- note added: "Bluetooth Serial"
- note added: "Channel Separation"
- note added: "Commutator"
- note added: "DC Power Jack"
- note added: "DC Restoration"
- note added: "DSR"
- note added: "DTR"
- note added: "Digital/Analog Voltage Domains"
- note added: "ECG"
- note added: "EN"
- note added: "Each module translates the 8V signals into 5V levels compatible with the Arduino ADC. The resistor divider has an attenuation of G = 50K / (30K + 50K) = 5 / 8. The op-amp is configured as a unity gain buffer, and provides a low output impedance to the ADC. IMPORTANT: If using alternate parts, ensure that the op amp for this stage is stable in a unity gain configuration\! The capacitor adds an opt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"
- note added: "Electrodes"
- note added: "GND"
- note added: "Gain & LPF"
- note added: "Gain (5X)"
- note added: "Gain is split across both sides of the high pass due to the DC offset on the inputs. To mitigate large input offsets, the IA gain should be reduced until the IA output is no longer saturated. The second stage gain should be increased to compensate for the reduced gain in the first stage. The Sallen-Key Lowpass Filter is designed for a cutoff frequency of 150 Hz and Q = 0.707 for a maximally flat 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"
- note added: "HPF"
- note added: "HPF (0.05 Hz)"
- note added: "ICG"
- note added: "ICG (con't)"
- note added: "ICG Channel -->"
- note added: "IOREF"
- note added: "Improved Howland Current Pump"
- note added: "Instrumentation Amplifier"
- note added: "Instrumentation Amplifier (Gain of 20X)"
- note added: "LED Drive, Clock Inversion"
- note added: "LPF & Gain"
- note added: "POWER"
- note added: "PPG"
- note added: "RESET"
- note added: "RX"
- note added: "Resp. Channel -->"
- note added: "Right Leg Drive"
- note added: "STATE"
- note added: "Sallen Key LPF (150 Hz, Q = 0.707)"
- note added: "Sallen-Key LPF"
- note added: "Sallen-Key LPF with optional gain"
- note added: "Sample & Hold"
- note added: "TX"
- note added: "The 8V regulator provides a stable 8V rail from an input source. The input source must be greater than 8V plus the transistor's collector-emitter drop. For the 2N2222 transistor, the max drop is 0.4V at 150 mA. By changing the gain resistors, the 8V regulator voltage can be modified and a different Zener diode can be used. The output voltage is calculated as follows: Vout = ((R11 + R19) / R11) * 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"
- note added: "VIN"
- note added: "Virtual Ground"

Commit message: Redesign
Parts:
- removed C2: 3.2u, SparkFun-Passives:CAPPTH1
- removed C22: (no value), SparkFun-Capacitors:CAPPTH1
- removed C3: 100nF, SparkFun-Passives:CAPPTH1
- removed C4: 220nF, SparkFun-Passives:CAPPTH1
- removed IC11, IC12, IC13: QUAD_OPAMPP, adafruit:QUAD_OPAMPP
- removed IC14, IC15: 4066N, 40xx:4066N
- removed R12, R2: 1M, adafruit:R-US_0204/5
- removed R13: 5M, adafruit:R-US_0204/5
- removed R28: 100K, adafruit:R-US_0204/5
- removed R3: 40K, adafruit:R-US_0204/5
- removed R4, R54, R55, R56, R57, R6: 10K, adafruit:R-US_0204/5
- removed R5: 5.1K, adafruit:R-US_0204/5
- removed R51, R52: 24.7K, adafruit:R-US_0204/5
- removed R53, R58: 1.3K, adafruit:R-US_0204/5
- removed R66: (no value), adafruit:R-US_0207/10
- removed R7, R8: 50K, adafruit:R-US_0204/5
- removed R86: (no value), rcl:R-US_0207/10
- removed SH1, SH2, SH3: SHORT, stanford_iot_research:SHORT
- removed T1, T2: 2N2222, adafruit:2N2222
- added C17, C18: (no value), SparkFun-Capacitors:CAPPTH1
- added CE1: 3.2u, SparkFun-Passives:CAPPTH1
- added CE2: 220nF, SparkFun-Passives:CAPPTH1
- added CE3: 100nF, SparkFun-Passives:CAPPTH1
- added D2, D4: 5V, diode:ZENER-DIODEZD-2.5
- added D3: 3V, diode:ZENER-DIODEZD-2.5
- added J10: POWER_JACKPTH, SparkFun-Connectors:POWER_JACKPTH
- added R44: (no value), rcl:R-US_0204/5
- added R45, R46, R47, R49, R50: 30K, adafruit:R-US_0204/5
- added R48, RE1, RE7: 50K, adafruit:R-US_0204/5
- added RE10, RE12, RE15, RE2, RE8, RE9: 10K, adafruit:R-US_0204/5
- added RE11, RE16: 1M, adafruit:R-US_0204/5
- added RE13: 40K, adafruit:R-US_0204/5
- added RE14: 5.1K, adafruit:R-US_0204/5
- added RE17: 5M, adafruit:R-US_0204/5
- added RE3, RE5: 1.3K, adafruit:R-US_0204/5
- added RE4, RE6: 24.7K, adafruit:R-US_0204/5
- C9: value 1nF -> (none); device SparkFun-Passives:CAPPTH1 -> SparkFun-Capacitors:CAPPTH1
- D1: value 5.1V -> 3V; device SparkFun-DiscreteSemi:DIODE-ZENERPTH -> diode:ZENER-DIODEZD-2.5
- IC1, IC3: value LMC660 -> QUAD_OPAMPP
- IC10: value QUAD_OPAMPP -> 4066N; device adafruit:QUAD_OPAMPP -> 40xx:4066N
- IC5: value 4066N -> QUAD_OPAMPP; device 40xx:4066N -> adafruit:QUAD_OPAMPP
- IC8: value LMC660 -> LM555N; device adafruit:QUAD_OPAMPP -> linear:LM555N
- IC9: value QUAD_OPAMPP -> LM555N; device adafruit:QUAD_OPAMPP -> linear:LM555N
- R1: value 10K -> (none); device adafruit:R-US_0204/5 -> rcl:R-US_0204/5
- R11: value 50K -> (none); device adafruit:R-US_0204/5 -> rcl:R-US_0207/10
- R14: value 30K -> (none); device adafruit:R-US_0204/5 -> rcl:R-US_0207/10
- R15, R17, R24: value 50K -> 30K
- R16: value 30K -> 50K
- R26: value 16K -> 30K
- R27: value 18K -> 50K
Connections:
- removed net AGND: C11.1, C12.1, C15.2, C23.2, C3.2, C32.1, C33.1, C37.2, C38.2, C9.2, IC12C.+IN, IC1D.+IN, IC5B.A, IC7A.+IN, J8.10, J8.12, J8.8, R10.1, R100.1, R2.1, R26.1, R31.1, R33.1, R4.1, R41.2, R57.2, R66.2, R68.1, R85.1, R86.1, R9.1, R92.1, R96.1, SH2.2, T3.E, T4.E
- removed net AVCC: IC1P.V+, R25.2, R29.2, SH1.2
- removed net AVSS: IC1P.V-, SH3.2
- removed net CLOCK1: C22.1, IC12A.OUT, R83.1, R87.2, R88.2
- removed net DGND: C1.2, C5.2, C6.2, C7.2, D1.A, IC2P.V-, IC4P.V-, J1.6, J1.7, J6.1, J6.2, J7.3, J9.GND, POWER.6, POWER.7, R11.1, R15.1, R17.1, R21.1, R22.1, R24.1, SH3.1
- removed net N$97: IC12A.+IN, R86.2, R87.1
- removed net VCC_4V: IC4B.-IN, SH2.1, T2.E
- removed net VCC_8V: R19.2, R20.2, SH1.1, T1.E, T2.C
- removed net VIN: IC4P.V+, J1.8, J9.PWR, POWER.8, R1.2, T1.C
- new net +8V: D1.C, IC10P.VDD, IC1P.V+, IC2P.V+, IC3P.V+, IC4P.V+, IC5P.V+, IC6P.V+, IC8.R, IC8.V+, IC9.R, IC9.V+, J1.8, J9.PWR, POWER.8, R11.2, R20.2, R25.2, R29.2, R87.2
- new net -8V: C1.1, C32.1, C33.2, C5.2, D3.C, IC10P.VSS, IC1P.V-, IC2P.V-, IC3P.V-, IC4P.V-, IC5P.V-, IC6P.V-, IC8.GND, IC9.GND, J10.GND
- new net 2.5V_BIAS: IC1B.-IN, IC1B.OUT, R16.1, R22.1, R27.1, R48.1
- new net 5V_ADCREF: IC1A.-IN, IC1A.OUT
- new net GND: C11.1, C12.1, C15.2, C18.2, C23.2, C37.2, C38.2, C6.2, C7.2, C9.2, CE3.2, D2.A, D4.A, IC10B.A, IC2D.+IN, IC3D.+IN, IC4B.+IN, IC7P.V-, J1.6, J1.7, J10.PWR, J6.1, J6.2, J7.3, J8.10, J8.12, J8.8, J9.GND, POWER.6, POWER.7, R1.1, R10.1, R100.1, R17.1, R23.1, R31.1, R33.1, R41.2, R44.1, R45.1, R49.1, R68.1, R85.1, R9.1, R92.1, R96.1, RE10.2, RE11.1, RE12.1, T3.E, T4.E
- new net N$54: IC7A.-IN, R17.2, R19.2
- new net N$56: IC7B.-IN, R23.2, R24.2
- new net N$58: C33.1, IC9.CV
- new net N$59: IC7C.-IN, R45.2, R46.2
- new net N$60: C18.1, IC7D.+IN, R47.2, R48.2
- new net N$61: IC7D.-IN, R49.2, R50.2
- new net N$63: C17.2, IC9.Q
- net 2KHZ_OSC: now also IC10C.C; no longer IC14B.C, IC6A.OUT, R27.2, R28.2
- net 30KHZ_OSC: now also C17.1, IC10A.C, R44.2, R83.1; no longer C22.2, IC5A.C, R66.1
- net ADC_ECG: now also IC7C.OUT, R46.1; no longer IC2C.-IN, IC2C.OUT
- net ADC_ICG: now also IC7A.OUT, R19.1; no longer IC2A.-IN, IC2A.OUT
- net ADC_PPG: now also IC7D.OUT, R50.1; no longer IC2D.-IN, IC2D.OUT
- net ADC_RESP: now also IC7B.OUT, R24.1; no longer IC2B.-IN, IC2B.OUT
- net ECG_E1: now also RE1.1; no longer R7.1
- net ECG_E2: now also RE7.1; no longer R8.1
- net ECG_E3: now also RE16.2, RE17.2; no longer R12.2, R13.2
- net ECG_OUT: now also CE2.2, IC1D.-IN, IC1D.OUT, R26.1; no longer C4.2, IC1B.-IN, IC1B.OUT, R18.1
- net ICG_DEMUX: now also IC4A.OUT; no longer IC12D.OUT
- net ICG_OUT: now also IC5A.OUT, R15.1; no longer IC11C.OUT, R14.1
- net N$10: now also D1.A, D2.C; no longer IC4A.OUT, T1.B
- net N$100: now also IC5D.+IN; no longer IC12B.+IN
- net N$101: now also IC3D.-IN; no longer IC12C.-IN
- net N$102: now also IC4A.+IN; no longer IC12D.+IN
- net N$103: now also IC5C.-IN; no longer IC11B.-IN
- net N$105: now also IC5B.-IN; no longer IC11A.-IN
- net N$107: now also IC5C.OUT; no longer IC11B.OUT
- net N$108: now also IC5A.+IN; no longer IC11C.+IN
- net N$109: now also IC5A.-IN; no longer IC11C.-IN
- net N$11: now also CE1.2, IC1C.+IN, RE11.2; no longer C2.2, IC1A.+IN, R2.2
- net N$12: now also CE3.1, IC1D.+IN, RE15.2; no longer C3.1, IC1B.+IN, R6.2
- net N$13: now also IC1C.OUT, RE13.2, RE14.1; no longer IC1A.OUT, R3.2, R5.1
- net N$14: now also CE2.1, RE14.2, RE15.1; no longer C4.1, R5.2, R6.1
- net N$15: now also IC2D.OUT, RE17.1; no longer IC1D.OUT, R13.1
- net N$16: now also IC2B.+IN, RE7.2; no longer IC9A.+IN, R8.2
- net N$2: now also IC1C.-IN, RE12.2, RE13.1; no longer IC1A.-IN, R3.1, R4.2
- net N$21: now also IC6C.+IN; no longer IC13B.+IN
- net N$23: now also IC3B.+IN; no longer IC10A.+IN
- net N$24: now also IC3D.OUT; no longer IC12C.OUT
- net N$25: now also IC3B.-IN; no longer IC10A.-IN
- net N$26: now also IC2D.-IN, RE16.1, RE3.1, RE5.2; no longer IC1D.-IN, R12.1, R53.1, R58.2
- net N$27: now also IC3B.OUT; no longer IC10A.OUT
- net N$28: now also IC1A.+IN, R20.1, R21.2; no longer C1.1, IC2A.+IN, R14.2, R15.2
- net N$29: now also IC8.DIS, R14.1; no longer C6.1, IC2C.+IN, R18.2, R22.2
- net N$3: now also IC1B.+IN, R1.2, R21.1; no longer C5.1, IC2B.+IN, R16.2, R17.2
- net N$30: now also C5.1, IC8.CV; no longer C7.1, IC2D.+IN, R23.2, R24.2
- net N$32: now also IC9.THR, IC9.TR, R87.1, R88.2; no longer C33.2, IC12A.-IN, R88.1
- net N$33: now also D3.A, D4.C; no longer IC4A.-IN, R11.2, R19.1
- net N$34: now also IC6A.-IN; no longer IC8C.-IN
- net N$35: now also IC10A.A; no longer IC5A.A
- net N$36: now also IC9.DIS, R88.1; no longer D1.C, IC4A.+IN, R1.1
- net N$37: now also IC10A.B, IC10B.B, IC4A.-IN; no longer IC12D.-IN, IC5A.B, IC5B.B
- net N$38: now also IC8.Q, R43.2, T4.B; no longer IC4B.+IN, R20.1, R21.2
- net N$39: now also IC6A.OUT; no longer IC8C.OUT
- net N$40: now also IC5B.+IN; no longer IC11A.+IN
- net N$41: now also C1.2, IC8.THR, IC8.TR, R11.1, R14.2; no longer IC4B.OUT, T2.B
- net N$42: now also IC6C.-IN; no longer IC13B.-IN
- net N$47: now also IC2B.-IN, RE5.1, RE6.1; no longer IC9A.-IN, R51.1, R58.1
- net N$48: now also C6.1, IC7A.+IN, R15.2, R16.2; no longer R43.2, T4.B
- net N$51: now also IC10B.C; no longer IC5B.C
- net N$53: now also IC6C.OUT; no longer IC13B.OUT
- net N$55: now also C7.1, IC7B.+IN, R18.2, R22.2; no longer C9.1, IC6A.-IN, R28.1
- net N$57: now also C9.1, IC7C.+IN, R27.2; no longer IC6A.+IN, R27.1
- net N$62: now also IC10C.A, IC10D.A, IC4B.OUT; no longer IC14B.A, IC15B.A, IC7A.OUT
- net N$64: now also IC4C.+IN; no longer IC7B.+IN
- net N$66: now also IC4C.-IN; no longer IC7B.-IN
- net N$67: now also IC4C.OUT; no longer IC7B.OUT
- net N$69: now also IC2B.OUT, RE6.2, RE8.1; no longer IC9A.OUT, R51.2, R56.1
- net N$7: now also IC6B.-IN; no longer IC13A.-IN
- net N$70: now also IC2C.+IN, RE10.1, RE8.2; no longer IC9B.+IN, R56.2, R57.1
- net N$71: now also IC2A.-IN, RE3.2, RE4.1; no longer IC1C.-IN, R52.1, R53.2
- net N$72: now also IC2A.OUT, RE2.1, RE4.2; no longer IC1C.OUT, R52.2, R54.1
- net N$73: now also IC2A.+IN, RE1.2; no longer IC1C.+IN, R7.2
- net N$74: now also IC3C.+IN; no longer IC10B.+IN
- net N$75: now also IC2C.-IN, RE2.2, RE9.1; no longer IC9B.-IN, R54.2, R55.1
- net N$76: now also IC3A.-IN; no longer IC3C.-IN
- net N$77: now also CE1.1, IC2C.OUT, RE9.2; no longer C2.1, IC9B.OUT, R55.2
- net N$78: now also IC3A.OUT; no longer IC3C.OUT
- net N$79: now also IC3A.+IN; no longer IC3C.+IN
- net N$80: now also IC3C.-IN; no longer IC10B.-IN
- net N$81: now also IC4D.+IN; no longer IC7C.+IN
- net N$84: now also IC3C.OUT; no longer IC10B.OUT
- net N$9: now also IC6B.OUT; no longer IC13A.OUT
- net N$95: now also IC5D.-IN; no longer IC12B.-IN
- net N$96: now also IC5C.+IN; no longer IC11B.+IN
- net PPG_DP: now also IC4B.-IN; no longer IC7A.-IN
- net PPG_IA_N: now also IC10D.B, IC6B.+IN; no longer IC13A.+IN, IC15B.B
- net PPG_IA_P: now also IC10C.B, IC6A.+IN; no longer IC14B.B, IC8C.+IN
- net PPG_LEDN: now also IC10D.C; no longer IC15B.C
- net PPG_OUT: now also IC4D.-IN, IC4D.OUT, R47.1; no longer IC7C.-IN, IC7C.OUT, R23.1
- net RESP_OUT: now also IC5B.OUT, R18.1; no longer IC11A.OUT, R16.1
- net V+: now also IC5D.OUT; no longer IC12B.OUT
- net VCC_5V: now also IC7P.V+; no longer IC2P.V+
Other:
- note added: "Bias Circuit"
- note added: "Power Rails +/- 8V"
- note removed: "8V Regulator"
- note removed: "AGND is NOT DGND\!\!"
- note removed: "Digital/Analog Voltage Domains"
- note removed: "Each module translates the 8V signals into 5V levels compatible with the Arduino ADC. The resistor divider has an attenuation of G = 50K / (30K + 50K) = 5 / 8. The op-amp is configured as a unity gain buffer, and provides a low output impedance to the ADC. IMPORTANT: If using alternate parts, ensure that the op amp for this stage is stable in a unity gain configuration\! The capacitor adds an opt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"
- note removed: "The 8V regulator provides a stable 8V rail from an input source. The input source must be greater than 8V plus the transistor's collector-emitter drop. For the 2N2222 transistor, the max drop is 0.4V at 150 mA. By changing the gain resistors, the 8V regulator voltage can be modified and a different Zener diode can be used. The output voltage is calculated as follows: Vout = ((R11 + R19) / R11) * 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"
- note removed: "Virtual Ground"

Commit message: Grouped items in layout
Parts:
- removed R10, R16, R20, R21, R22, R27, R48, R9: 50K, adafruit:R-US_0204/5
- removed R100, R11, R14, R87, R88, R91, R99: (no value), rcl:R-US_0207/10
- removed R15, R17, R18, R19, R23, R24, R26, R45, R46, R47, R49, R50: 30K, adafruit:R-US_0204/5
- removed R29: 120-320, adafruit:R-US_0204/5
- removed R30: 220K, adafruit:R-US_0204/5
- removed R31: 160K, adafruit:R-US_0204/5
- removed R32: 500K, adafruit:R-US_0204/5
- removed R33: 1K-6K, adafruit:R-US_0204/5
- removed R34: 2.4K, adafruit:R-US_0204/5
- removed R35: 3.9K, adafruit:R-US_0204/5
- removed R36, R37: 4.99K, adafruit:R-US_0204/5
- removed R38, R39, R40, R41: 9.53K, adafruit:R-US_0204/5
- removed R42: (no value), adafruit:R-US_0204/5
- removed R43, R61, R62, R63, R64: 10K, adafruit:R-US_0204/5
- removed R44: (no value), rcl:R-US_0204/5
- removed R59, R60: 24.7K, adafruit:R-US_0204/5
- removed R65: 1.3K, adafruit:R-US_0204/5
- removed R67, R68, R70, R71, R72, R78, R82, R83, R85, R92, R93, R94, R95, R96, R97, R98: (no value), adafruit:R-US_0207/10
- added C19: 1uF, adafruit:CPOL-USE2-5
- added C2, C3, C4: 100uF, SparkFun-Passives:CAP_POLPTH1
- added CA1, CA2, CA3, CA4, CI6, CP1, CP2: (no value), SparkFun-Capacitors:CAPPTH1
- added CP3: 22pF, SparkFun-Passives:CAPPTH1
- added CP4, CP5: 100nF, SparkFun-Passives:CAPPTH1
- added CP6: 10uF, SparkFun-Passives:CAPPTH1
- added CP7: 10nF, SparkFun-Passives:CAPPTH1
- added CP8: 1uF, SparkFun-Passives:CAPPTH1
- added CP9: 4.3uF, SparkFun-Passives:CAPPTH1
- added R2, R3, RA10, RA14, RA2, RA6, RI1, RI34: 50K, resistor:R-US_0207/10
- added RA1, RA11, RA12, RA13, RA15, RA16, RA3, RA4, RA5, RA7, RA8, RA9: 30K, resistor:R-US_0207/10
- added RI10, RI11, RI12, RI13, RI14, RI15, RI16, RI17, RI18, RI19, RI20, RI21, RI23, RI24, RI25, RI26, RI27, RI28, RI29, RI30, RI31, RI32, RI33, RP1, RP2, RP9: (no value), resistor:R-US_0207/10
- added RI2, RI3, RI7, RI8, RP4: 10K, resistor:R-US_0207/10
- added RI4, RI6: 24.7K, resistor:R-US_0207/10
- added RI5: 1.3K, resistor:R-US_0207/10
- added RP10, RP8: 4.99K, resistor:R-US_0207/10
- added RP11, RP12, RP6, RP7: 9.53K, resistor:R-US_0207/10
- added RP13: 160K, resistor:R-US_0207/10
- added RP14: 1K-6K, resistor:R-US_0207/10
- added RP15: 500K, resistor:R-US_0207/10
- added RP16: 2.4K, resistor:R-US_0207/10
- added RP17: 3.9K, resistor:R-US_0207/10
- added RP3: 120-320, resistor:R-US_0207/10
- added RP5: 220K, resistor:R-US_0207/10
- C1, C17, C18, C5, C6, C7, C9: value (none) -> 100uF; device SparkFun-Capacitors:CAPPTH1 -> SparkFun-Passives:CAP_POLPTH1
- C10: value 22pF -> 100uF; device SparkFun-Passives:CAPPTH1 -> SparkFun-Passives:CAP_POLPTH1
- C11, C12: value 100nF -> 100uF; device SparkFun-Passives:CAPPTH1 -> SparkFun-Passives:CAP_POLPTH1
- C13: value 10uF -> 100uF; device SparkFun-Passives:CAPPTH1 -> SparkFun-Passives:CAP_POLPTH1
- C14: value 10nF -> 100uF; device SparkFun-Passives:CAPPTH1 -> SparkFun-Passives:CAP_POLPTH1
- C15: value 1uF -> 100uF; device SparkFun-Passives:CAPPTH1 -> SparkFun-Passives:CAP_POLPTH1
- C16: value 4.3uF -> 100uF; device SparkFun-Passives:CAPPTH1 -> SparkFun-Passives:CAP_POLPTH1
- C8: value 1uF -> 100uF; device adafruit:CPOL-USE2-5 -> SparkFun-Passives:CAP_POLPTH1
- D1, D2, D3, D4: device diode:ZENER-DIODEZD-2.5 -> diode:ZENER-DIODEZD-10
- R1: device rcl:R-US_0204/5 -> resistor:R-US_0207/10
- RE1, RE10, RE11, RE12, RE13, RE14, RE15, RE16, RE17, RE2, RE3, RE4, RE5, RE6, RE7, RE8, RE9: device adafruit:R-US_0204/5 -> resistor:R-US_0207/10
- renumbered C20 to CI1, C21 to CI2, C23 to CI9, C24 to CI3, C29 to CI7, C32 to CI5, C33 to CI4, C34 to CI8, C35 to CI10, C36 to CI12, C37 to CI11, C38 to CI13, R25 to RI22, R69 to RI9
Connections:
- net N$51 renamed RI13
- new net N$51: RI13.1, T3.B
- net +8V: now also C1.+, C2.+, C3.+, C4.+, C5.+, C6.+, C7.+, C8.+, C9.+, R3.2, RI14.2, RP2.2, RP3.2; no longer R11.2, R20.2, R29.2, R87.2
- net -8V: now also C10.-, C11.-, C12.-, C13.-, C14.-, C15.-, C16.-, C17.-, C18.-, CP1.2, CP2.1; no longer C1.1, C5.2
- net 2.5V_BIAS: now also RA10.1, RA14.1, RA2.1, RA6.1; no longer R16.1, R22.1, R27.1, R48.1
- net 2KHZ_OSC: now also IC8.Q, RP4.1; no longer R43.1
- net 30KHZ_OSC: now also CI6.1, RI13.2, RI16.2, RI20.1; no longer C17.1, R44.2, R83.1, T3.B
- net ADC_ECG: now also RA12.1; no longer R46.1
- net ADC_ICG: now also RA4.1; no longer R19.1
- net ADC_PPG: now also RA16.1; no longer R50.1
- net ADC_RESP: now also RA8.1; no longer R24.1
- net ECG_OUT: now also RA9.1; no longer R26.1
- net ELECTRODE3: now also RI18.2, RI19.1; no longer R78.1, R91.2
- net GND: now also C1.-, C10.+, C11.+, C12.+, C13.+, C14.+, C15.+, C16.+, C17.+, C18.+, C2.-, C3.-, C4.-, C5.-, C6.-, C7.-, C8.-, C9.-, CA1.2, CA2.2, CA3.2, CA4.2, CP4.1, CP5.1, CP8.2, RA11.1, RA15.1, RA3.1, RA7.1, RI1.1, RI16.1, RI17.1, RI24.1, RI26.1, RI29.1, RI33.1, RI34.1, RP12.2, RP13.1, RP14.1; no longer C11.1, C12.1, C15.2, C18.2, C6.2, C7.2, C9.2, R10.1, R100.1, R17.1, R23.1, R31.1, R33.1, R41.2, R44.1, R45.1, R49.1, R68.1, R85.1, R9.1, R92.1, R96.1
- net ICG_DEMUX: now also RI12.2, RI23.1, RI31.1; no longer R67.1, R72.2, R95.1
- net ICG_OUT: now also RA1.1, RI30.2; no longer R15.1, R99.2
- net N$100: now also RI17.2, RI18.1; no longer R85.2, R91.1
- net N$102: now also RI10.2, RI12.1; no longer R70.2, R72.1
- net N$103: now also RI25.1, RI26.2; no longer R92.2, R93.1
- net N$105: now also RI32.1, RI33.2; no longer R96.2, R97.1
- net N$106: now also RI27.2, RI28.1; no longer R94.2, R98.1
- net N$107: now also RI25.2, RI27.1; no longer R93.2, R94.1
- net N$108: now also RI28.2; no longer R98.2
- net N$109: now also RI29.2, RI30.1; no longer R100.2, R99.1
- net N$110: now also RI23.2; no longer R67.2
- net N$21: now also RP11.2, RP12.1; no longer R40.2, R41.1
- net N$23: now also RI34.2; no longer R10.2
- net N$24: now also RI8.2; no longer R64.2
- net N$25: now also RI5.1, RI6.1; no longer R59.1, R65.1
- net N$27: now also RI6.2, RI7.1; no longer R59.2, R63.1
- net N$28: now also R2.2, R3.1; no longer R20.1, R21.2
- net N$29: now also RP1.1; no longer R14.1
- net N$3: now also R2.1; no longer R21.1
- net N$30: now also CP1.1; no longer C5.1
- net N$32: now also RI14.1, RI15.2; no longer R87.1, R88.2
- net N$34: now also RP8.1, RP9.2; no longer R37.1, R42.2
- net N$35: now also RI11.2; no longer R71.2
- net N$36: now also RI15.1; no longer R88.1
- net N$38: now also RP4.2; no longer IC8.Q, R43.2
- net N$39: now also RP6.1, RP8.2; no longer R37.2, R38.1
- net N$40: now also RI31.2; no longer R95.2
- net N$41: now also CP2.2, RP1.2, RP2.1; no longer C1.2, R11.1, R14.2
- net N$42: now also RP6.2, RP7.1; no longer R38.2, R39.1
- net N$48: now also CA1.1, RA1.2, RA2.2; no longer C6.1, R15.2, R16.2
- net N$53: now also CP6.1, RP7.2; no longer C13.1, R39.2
- net N$54: now also RA3.2, RA4.2; no longer R17.2, R19.2
- net N$55: now also CA2.1, RA5.2, RA6.2; no longer C7.1, R18.2, R22.2
- net N$56: now also RA7.2, RA8.2; no longer R23.2, R24.2
- net N$57: now also CA3.1, RA10.2, RA9.2; no longer C9.1, R26.2, R27.2
- net N$59: now also RA11.2, RA12.2; no longer R45.2, R46.2
- net N$6: now also C19.-; no longer C8.-
- net N$60: now also CA4.1, RA13.2, RA14.2; no longer C18.1, R47.2, R48.2
- net N$61: now also RA15.2, RA16.2; no longer R49.2, R50.2
- net N$62: now also CP3.1, RP5.2; no longer C10.1, R30.2
- net N$63: now also CI6.2; no longer C17.2
- net N$64: now also CP6.2, RP13.2; no longer C13.2, R31.2
- net N$66: now also CP7.2, RP14.2, RP15.1; no longer C14.2, R32.1, R33.2
- net N$67: now also CP7.1, RP15.2, RP16.1; no longer C14.1, R32.2, R34.1
- net N$68: now also CP9.1, RP16.2, RP17.1; no longer C16.1, R34.2, R35.1
- net N$7: now also RP10.1, RP9.1; no longer R36.1, R42.1
- net N$74: now also RI7.2, RI8.1; no longer R63.2, R64.1
- net N$76: now also RI4.1, RI5.2; no longer R60.1, R65.2
- net N$78: now also RI2.1, RI4.2; no longer R60.2, R61.1
- net N$79: now also RI1.2; no longer R9.2
- net N$80: now also RI2.2, RI3.1; no longer R61.2, R62.1
- net N$81: now also CP8.1, RP17.2; no longer C15.1, R35.2
- net N$84: now also RI10.1, RI11.1, RI3.2; no longer R62.2, R70.1, R71.1
- net N$9: now also RP10.2, RP11.1; no longer R36.2, R40.1
- net N$95: now also RI20.2, RI21.1; no longer R82.1, R83.2
- net N$96: now also RI24.2; no longer R68.2
- net PPG_DP: now also CP3.2, RP5.1; no longer C10.2, R30.1
- net PPG_IA_N: now also CP5.2; no longer C11.2
- net PPG_IA_P: now also CP4.2; no longer C12.2
- net PPG_LEDP: now also RP3.1; no longer R29.1
- net PPG_OUT: now also CP9.2, RA13.1; no longer C16.2, R47.1
- net RESET: now also C19.+; no longer C8.+
- net RESP_OUT: now also RA5.1, RI32.2; no longer R18.1, R97.2
- net V+: now also RI19.2, RI21.2; no longer R78.2, R82.2

Commit message: Revision 1
Parts:
- removed C14, C6, C9: 100uF, SparkFun-Passives:CAP_POLPTH1
- removed DIGITAL2: (no value), SmartPrj:PINHD-1X10TH
- removed J2: (no value), pinhead:PINHD-1X5
- removed J4, POWER: (no value), SmartPrj:PINHD-1X8TH
- removed J5: (no value), pinhead:PINHD-1X1
- added R4: 100, resistor:R-US_0207/10
- added RP18: 10K, resistor:R-US_0207/10
Connections:
- net PPG_IA_N renamed PPG_IAN
- net PPG_IA_P renamed PPG_IAP
- removed net CLK: DIGITAL1.4, J4.4
- removed net DIN: DIGITAL1.8, J4.8
- removed net N$1: DIGITAL2.7, J3.7
- removed net N$17: DIGITAL2.2, J3.2
- removed net N$18: J1.1, POWER.1
- removed net N$19: J1.2, POWER.2
- removed net N$20: J1.4, POWER.4
- removed net N$22: DIGITAL1.6, J4.6
- removed net N$31: DIGITAL1.3, J4.3
- removed net N$4: DIGITAL1.7, J4.7
- removed net N$43: DIGITAL2.3, J3.3
- removed net N$44: DIGITAL2.4, J3.4
- removed net N$45: DIGITAL2.5, J3.5
- removed net N$46: DIGITAL2.6, J3.6
- removed net N$49: DIGITAL2.9, J3.9
- removed net N$5: DIGITAL1.5, J4.5
- removed net N$50: DIGITAL2.10, J3.10
- removed net N$52: ANALOG.6, J5.1
- removed net N$8: ANALOG.5, J2.5
- removed net VB: DIGITAL2.1, J3.1
- new net N$10000: IC8.Q, RP4.1
- new net N$65: IC10D.C, R4.2
- net +8V: no longer C6.+, C9.+, POWER.8
- net -8V: no longer C14.-
- net 2KHZ_OSC: now also RP18.2, RP4.2, T4.B; no longer IC10C.C, IC8.Q, RP4.1
- net 5V_ADCREF: now also J3.8
- net ADC_ECG: no longer J2.2
- net ADC_ICG: no longer J2.4
- net ADC_PPG: no longer J2.1
- net ADC_RESP: no longer J2.3
- net GND: no longer C14.+, C6.-, C9.-, POWER.6, POWER.7
- net N$38: now also IC10C.C, RP18.1; no longer RP4.2, T4.B
- net PPG_LEDN: now also R4.1; no longer IC10D.C
- net RESET: no longer POWER.3
- net RX: no longer J4.1
- net TX: no longer J4.2
- net VCC_5V: no longer DIGITAL2.8, J3.8, POWER.5
