File: bioshield.sch (EAGLE design)
At the start: 159 parts, among them IC1 QUAD_OPAMPP, IC10 4066N, IC2 QUAD_OPAMPP, IC3 QUAD_OPAMPP, IC4 QUAD_OPAMPP, IC5 QUAD_OPAMPP, IC6 QUAD_OPAMPP, IC7 QUAD_OPAMPP, IC8 LM555N, IC9 LM555N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

Commit message: Pre-assembly
Parts:
- R1: value (none) -> 25K
- R2, RA10, RA14, RA2, RA6: value 50K -> 25K
- R3: value 50K -> 30K
- RA1, RA11, RA13, RA15, RA3, RA5, RA7, RA9: value 30K -> 80K
- RA12, RA16, RA4, RA8: value 30K -> 25K
Changed lines of the file:
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@@
 <part name="IC4" library="adafruit" deviceset="QUAD_OPAMP" device="P"/>
 <part name="IC5" library="adafruit" deviceset="QUAD_OPAMP" device="P"/>
-<part name="R3" library="resistor" deviceset="R-US_" device="0207/10" value="50K"/>
-<part name="R2" library="resistor" deviceset="R-US_" device="0207/10" value="50K"/>
+<part name="R3" library="resistor" deviceset="R-US_" device="0207/10" value="30K"/>
+<part name="R2" library="resistor" deviceset="R-US_" device="0207/10" value="25K"/>
 <part name="GND9" library="SparkFun-Aesthetics" deviceset="DGND" device=""/>
 <part name="D1" library="diode" deviceset="ZENER-DIODE" device="ZD-10" value="3V"/>
@@
 <part name="D3" library="diode" deviceset="ZENER-DIODE" device="ZD-10" value="3V"/>
 <part name="D4" library="diode" deviceset="ZENER-DIODE" device="ZD-10" value="5V"/>
-<part name="R1" library="resistor" deviceset="R-US_" device="0207/10"/>
+<part name="R1" library="resistor" deviceset="R-US_" device="0207/10" value="25K"/>
 <part name="SUPPLY3" library="supply2" deviceset="+8V" device=""/>
 <part name="SUPPLY5" library="supply2" deviceset="-8V" device=""/>
@@
 <part name="SUPPLY23" library="supply2" deviceset="+8V" device=""/>
 <part name="SUPPLY24" library="supply2" deviceset="-8V" device=""/>
-<part name="RA1" library="resistor" deviceset="R-US_" device="0207/10" value="30K"/>
-<part name="RA2" library="resistor" deviceset="R-US_" device="0207/10" value="50K"/>
+<part name="RA1" library="resistor" deviceset="R-US_" device="0207/10" value="80K"/>
+<part name="RA2" library="resistor" deviceset="R-US_" device="0207/10" value="25K"/>
 <part name="CA1" library="SparkFun-Capacitors" deviceset="CAP" device="PTH1"/>
 <part name="IC7" library="adafruit" deviceset="QUAD_OPAMP" device="P"/>
-<part name="RA3" library="resistor" deviceset="R-US_" device="0207/10" value="30K"/>
-<part name="RA4" library="resistor" deviceset="R-US_" device="0207/10" value="30K"/>
-<part name="RA5" library="resistor" deviceset="R-US_" device="0207/10" value="30K"/>
-<part name="RA6" library="resistor" deviceset="R-US_" device="0207/10" value="50K"/>
+<part name="RA3" library="resistor" deviceset="R-US_" device="0207/10" value="80K"/>
+<part name="RA4" library="resistor" deviceset="R-US_" device="0207/10" value="25K"/>
+<part name="RA5" library="resistor" deviceset="R-US_" device="0207/10" value="80K"/>
+<part name="RA6" library="resistor" deviceset="R-US_" device="0207/10" value="25K"/>
 <part name="CA2" library="SparkFun-Capacitors" deviceset="CAP" device="PTH1"/>
-<part name="RA7" library="resistor" deviceset="R-US_" device="0207/10" value="30K"/>
-<part name="RA8" library="resistor" deviceset="R-US_" device="0207/10" value="30K"/>
-<part name="RA9" library="resistor" deviceset="R-US_" device="0207/10" value="30K"/>
-<part name="RA10" library="resistor" deviceset="R-US_" device="0207/10" value="50K"/>
+<part name="RA7" library="resistor" deviceset="R-US_" device="0207/10" value="80K"/>
+<part name="RA8" library="resistor" deviceset="R-US_" device="0207/10" value="25K"/>
+<part name="RA9" library="resistor" deviceset="R-US_" device="0207/10" value="80K"/>
+<part name="RA10" library="resistor" deviceset="R-US_" device="0207/10" value="25K"/>
 <part name="CA3" library="SparkFun-Capacitors" deviceset="CAP" device="PTH1"/>
-<part name="RA11" library="resistor" deviceset="R-US_" device="0207/10" value="30K"/>
-<part name="RA12" library="resistor" deviceset="R-US_" device="0207/10" value="30K"/>
-<part name="RA13" library="resistor" deviceset="R-US_" device="0207/10" value="30K"/>
-<part name="RA14" library="resistor" deviceset="R-US_" device="0207/10" value="50K"/>
+<part name="RA11" library="resistor" deviceset="R-US_" device="0207/10" value="80K"/>
+<part name="RA12" library="resistor" deviceset="R-US_" device="0207/10" value="25K"/>
+<part name="RA13" library="resistor" deviceset="R-US_" device="0207/10" value="80K"/>
+<part name="RA14" library="resistor" deviceset="R-US_" device="0207/10" value="25K"/>
 <part name="CA4" library="SparkFun-Capacitors" deviceset="CAP" device="PTH1"/>
-<part name="RA15" library="resistor" deviceset="R-US_" device="0207/10" value="30K"/>
-<part name="RA16" library="resistor" deviceset="R-US_" device="0207/10" value="30K"/>
+<part name="RA15" library="resistor" deviceset="R-US_" device="0207/10" value="80K"/>
+<part name="RA16" library="resistor" deviceset="R-US_" device="0207/10" value="25K"/>
 <part name="SUPPLY10" library="supply2" deviceset="-8V" device=""/>
 <part name="SUPPLY11" library="supply2" deviceset="+8V" device=""/>
